File: kicad/power-supply/power-supply.kicad_sch (KiCad schematic)
At the start: 104 parts, among them J1 Conn_01x03, Q1 NMOS, Q2 NMOS, Q3 NMOS, Q4 NMOS, U1 TPS568230RJER, U2 TPS568230RJER, U3 INA226, U4 HY2120, U5 HY2213-BB3A, U6 HY2213-BB3A, U7 TPS568230RJER

Commit message: completed power board
Parts:
- added C45, C46: 22uF, symbol Device:C
- added C47: 100 nF, symbol Device:C_Small
- added C48: 100n, symbol Device:C_Small
- added C49, C50, C52: 1u, symbol Device:C_Small
- added C51: 100nf, symbol Device:C_Small
- added D1, D2, D3, D4, D5: LED, symbol Device:LED
- added F1: Fuse, symbol Device:Fuse
- added IP1: IP2368, symbol IP2368:IP2368
- added J2: USB_C_Receptacle_USB2.0_16P, symbol Connector:USB_C_Receptacle_USB2.0_16P
- added L3: 10uH, symbol Device:L
- added Q5, Q6, Q7, Q8, Q9: NMOS, symbol Simulation_SPICE:NMOS
- added R38, R39, R45: 1K, symbol Device:R
- added R40, R41: 5m, symbol Device:R
- added R42: 6.2k, symbol Device:R
- added R43: 10k, symbol Device:R
- added R44: 27K, symbol Device:R
- added R46: 12.4K, symbol Device:R
- added SW1: SW_SPST, symbol Switch:SW_SPST
- added TH1: Thermistor_NTC, symbol Device:Thermistor_NTC
- added TP1, TP10, TP2, TP3, TP4, TP5, TP6, TP7, TP8, TP9: TestPoint, symbol Connector:TestPoint
Connections:
- net +3V3: now also TP8.1
- net +5V: now also TP7.1
- net BAT+: now also F1.2, IP1.25 (CSN2), IP1.27 (BAT), R41.2, TP1.1; no longer BT1.1 (+), BT2.1 (+), BT3.1 (+), BT4.1 (+), R13.2, R14.2
- net BAT-: now also TP4.1
- net GND: now also C45.2, C46.2, C49.2, C50.2, C51.2, C52.1, D1.1 (K), D2.2 (A), D3.1 (K), D4.2 (A), D5.1 (K), IP1.11 (AGND), IP1.30 (AGND), IP1.4 (LED3), IP1.49 (EPAD), J2.A1 (GND), J2.A12 (GND), J2.B1 (GND), J2.B12 (GND), J2.S1 (SHIELD), Q7.3 (S), Q9.3 (S), R42.1, R43.1, R44.2, R46.1, SW1.2 (B), TH1.2, TP2.1; no longer R24.1, R27.1, R4.1
- net PBS+: now also TP5.1
- net VOUT-1: now also TP6.1
- net at J1.1 (Pin_1), J1.3 (Pin_3), R34.1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: now also TP9.1
- net at J1.2 (Pin_2), R35.1, U3.5 (SCL): now also TP10.1
- new net: IP1.5 (HLED), R45.1
- new net: D5.2 (A), R45.2
- new net: C47.1, IP1.18 (LX1), L3.2, Q6.3 (S), Q7.1 (D)
- new net: IP1.19 (LG1), Q7.2 (G)
- new net: C48.1, IP1.21 (LX2), L3.1, Q8.3 (S), Q9.1 (D)
- new net: C45.1, C46.1, IP1.8 (VBUS), J2.A4 (VBUS), J2.A9 (VBUS), J2.B4 (VBUS), J2.B9 (VBUS), Q5.1 (D)
- new net: C52.2, IP1.12 (VI0)
- new net: IP1.10 (VBUS_1), IP1.13 (CSP1), Q5.3 (S), R40.1
- new net: IP1.14 (CSN1), IP1.15 (PCIN), Q6.1 (D), R40.2
- new net: BT1.1 (+), BT2.1 (+), BT3.1 (+), BT4.1 (+), F1.1, R13.2, R14.2, TP3.1
- new net: IP1.35 (VSET), R43.2
- new net: IP1.42 (LED2), R39.1
- new net: D3.2 (A), D4.1 (K), R39.2
- new net: C51.1, IP1.37 (NTC), TH1.1
- new net: IP1.33 (BAT_NUM), R42.2
- new net: IP1.26 (CSP2), Q8.1 (D), R41.1
- new net: IP1.36 (ISET), R44.1
- new net: D1.2 (A), D2.1 (K), R38.1
- new net: IP1.34 (FCAP), R46.2
- new net: C50.1, IP1.29 (VCC5V)
- new net: C47.2, IP1.17 (BST1)
- new net: IP1.16 (HG1), Q6.2 (G)
- new net: IP1.23 (HG2), Q8.2 (G)
- new net: IP1.43 (LED1), R38.2
- new net: IP1.20 (LG2), Q9.2 (G)
- new net: IP1.9 (VBUSG), Q5.2 (G)
- new net: C48.2, IP1.22 (BST2)
- new net: C49.1, IP1.32 (VCCIO)
- new net CC1: IP1.41 (CC1), J2.A5 (CC1)
- new net CC2: IP1.38 (CC2), J2.B5 (CC2)
- new net DMC: IP1.39 (DPC), J2.A6 (D+), J2.B6 (D+)
- new net DPC: IP1.40 (DMC), J2.A7 (D-), J2.B7 (D-)
- new net EN: R24.1, R27.1, R4.1, SW1.1 (A)
- no-connect marks 0 -> 4
Other:
- note added: "10K"
- note added: "CIPHER - by ARYAN-GIT-BYTE"
- note added: "NMOS = HUASHUO HSBA4094"
- note added: "PLACEHOLDER FOR CONNECTORS (TO BE PLACED)"
- note added: "R42- 6.2K , CONFIGURE IT FOR 2S R32 - 10K, SETS MAX CHARGE VOLTAGE AS 4.2V FOR 1 CELL, 8.4V TOTAL R44 - 27K , SETS THE PD INPUT POWER LIMIT TO 100W R43 - 12.4K, TELLS THAT THE TOTAL CURRENT OF 4P CELLS ARE 10,000 mAh"
- note added: "TYPE-C CHARGER"
- note removed: "NMOS = AOD4184-XBLW-40V 60A"

Commit message: made overall schematic
Parts:
- added J6, J7: Conn_01x02, symbol Connector_Generic:Conn_01x02
Connections:
- net +3V3: now also J7.1 (Pin_1)
- net GND: now also J6.2 (Pin_2), J7.2 (Pin_2)
- net VOUT-1 renamed 5V_OUT
- net 5V_OUT: now also J6.1 (Pin_1)
Other:
- note removed: "PLACEHOLDER FOR CONNECTORS (TO BE PLACED)"

Commit message: finally completed the schematic
Parts:
- removed IP1: IP2368, symbol IP2368:IP2368
- removed U4: HY2120, symbol HY2120:_1
- removed U5, U6: HY2213-BB3A, symbol HY2120:HY2213
- added IP2: ~, symbol IP2368:IP2368
- added J15: Conn_01x02, symbol Connector_Generic:Conn_01x02
- added U26: HY2120, symbol HY2120:HY2120
- added U7, U9: HY2213-BB3A, symbol HY2213:HY2213
- R30: renamed from R3; value 220K -> 160K
- renumbered BT1 to BT2, BT2 to BT3, BT3 to BT4, BT4 to BT5, BT5 to BT6, BT6 to BT7, BT7 to BT8, BT8 to BT9, C29 to C10, C34 to C11, C44 to C12, C30 to C13, C31 to C14, C32 to C15, C40 to C16, C35 to C17, C36 to C18, C37 to C19, C38 to C20, C39 to C21, C41 to C22, C33 to C23, C1 to C24, C2 to C25, C3 to C26, C4 to C27, C5 to C28, C6 to C29, C7 to C30, C8 to C31, C9 to C32, C10 to C33, C11 to C34, C12 to C35, C13 to C36, C51 to C37, C45 to C38, C46 to C39, C49 to C40, C50 to C41, C14 to C42, C15 to C43, C52 to C44, C16 to C45, C17 to C46, C18 to C47, C19 to C48, C20 to C49, C21 to C50, C22 to C51, C23 to C52, C24 to C53, C42 to C54, C43 to C55, C48 to C56, C47 to C57, C25 to C6, C26 to C7, C27 to C8, C28 to C9, D1 to D3, D2 to D4, D3 to D5, D4 to D6, D5 to D7, J6 to J14, J7 to J16, J1 to J17, J2 to J18, L4 to L1, L1 to L2, L2 to L3, L3 to L4, Q3 to Q1, Q1 to Q3, Q8 to Q6, Q6 to Q7, Q9 to Q8, Q7 to Q9, R15 to R10, R16 to R11, R21 to R12, R32 to R13, R33 to R14, R35 to R15, R36 to R16, R34 to R17, R17 to R18, R22 to R19, R24 to R20, R18 to R21, R23 to R22, R37 to R23, R19 to R24, R20 to R25, R1 to R26, R38 to R27, R39 to R28, R2 to R29, R4 to R31, R5 to R32, R6 to R33, R45 to R34, R44 to R35, R7 to R36, R43 to R37, R8 to R38, R46 to R39, R42 to R40, R9 to R41, R41 to R42, R40 to R43, R25 to R44, R26 to R45, R27 to R46, R28 to R47, R29 to R48, R30 to R49, R14 to R5, R31 to R50, R10 to R6, R13 to R7, R11 to R8, R12 to R9, TP5 to TP10, TP7 to TP11, TP8 to TP12, TP1 to TP3, TP3 to TP4, TP2 to TP5, TP4 to TP6, TP6 to TP7, TP9 to TP8, TP10 to TP9, U7 to U10, U3 to U11, U1 to U12, U2 to U13
Connections:
- net BAT+: now also IP2.25 (CSN2), IP2.27 (BAT)
- net BAT-: now also U26.6 (VSS), U9.3 (VSS)
- net BAT_MID: now also U7.3 (VSS)
- net CC1: now also IP2.41 (CC1)
- net CC2: now also IP2.38 (CC2)
- net DMC: now also IP2.39 (DPC)
- net DPC: now also IP2.40 (DMC)
- net GND: now also IP2.11 (AGND), IP2.30 (AGND), IP2.4 (LED3), IP2.49 (EPAD), J15.2 (Pin_2)
- net at R34.1: now also IP2.5 (HLED)
- net at Q2.2 (G): now also U26.1 (OD)
- net at Q3.2 (G): now also U26.2 (OC)
- net at R9.2: now also U26.3 (CS)
- net at C7.1, R8.2: now also U26.4 (VC)
- net at C6.2, R6.2: now also U26.5 (VDD)
- net at C57.1, L4.2, Q7.3 (S)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: now also IP2.18 (LX1)
- net at Q9.2 (G): now also IP2.19 (LG1)
- net at C56.1, L4.1, Q6.3 (S)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: now also IP2.21 (LX2)
- net at C38.1, C39.1, J18.A4 (VBUS)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: now also IP2.8 (VBUS)
- net at C44.2: now also IP2.12 (VI0)
- net at Q5.3 (S), R43.1: now also IP2.10 (VBUS_1), IP2.13 (CSP1)
- net at Q7.1 (D), R43.2: now also IP2.14 (CSN1), IP2.15 (PCIN)
- net at R37.2: now also IP2.35 (VSET)
- net at R28.1: now also IP2.42 (LED2)
- net at C37.1, TH1.1: now also IP2.37 (NTC)
- net at R40.2: now also IP2.33 (BAT_NUM)
- net at C9.1, R11.1: now also U9.2 (VDD)
- net at Q6.1 (D), R42.1: now also IP2.26 (CSP2)
- net at R35.1: now also IP2.36 (ISET)
- net at C8.1, R7.1: now also U7.2 (VDD)
- net at Q4.2 (G): now also U9.6 (OUT)
- net at R39.2: now also IP2.34 (FCAP)
- net at Q1.2 (G): now also U7.6 (OUT)
- net at C41.1: now also IP2.29 (VCC5V)
- net at C57.2: now also IP2.17 (BST1)
- net at Q7.2 (G): now also IP2.16 (HG1)
- net at Q6.2 (G): now also IP2.23 (HG2)
- net at R27.2: now also IP2.43 (LED1)
- net at Q8.2 (G): now also IP2.20 (LG2)
- net at Q5.2 (G): now also IP2.9 (VBUSG)
- net at C56.2: now also IP2.22 (BST2)
- net at C40.1: now also IP2.32 (VCCIO)
- net +3V3 renamed 3V3_OUT
- net +5V renamed 3V8_OUT
- net 3V8_OUT: now also J15.1 (Pin_1)
- net PBS+ renamed VBAT
- no-connect marks 4 -> 13
Other:
- note added: "4.2V@8A PEAK CHANNEL - 2"
- note added: "CONNECTORS"
- note removed: "5V@8A PEAK CHANNEL - 2"
- moved on the sheet: J14, J16

Commit message: DOCUMENTED Till the Navigation board
Parts:
- added J3, J4, J6, J8: Conn_01x02, symbol Connector_Generic:Conn_01x02
- added J58: Conn_01x03, symbol Connector_Generic:Conn_01x03
Connections:
- net 3V3_OUT: now also J4.1 (Pin_1)
- net 5V_OUT: now also J3.1 (Pin_1), J58.1 (Pin_1), J6.1 (Pin_1), J8.1 (Pin_1)
- net GND: now also J3.2 (Pin_2), J4.2 (Pin_2), J58.2 (Pin_2), J6.2 (Pin_2), J8.2 (Pin_2)
- net VBAT: now also J58.3 (Pin_3)
Other:
- note added: "JST-XH CONNECTOR TO CONNECT TO THE GPIO BREAKOUT BOARD"
- note added: "JST-XH CONNECTOR TO CONNECT TO THE NAVIGATION BOARD"
- note added: "JST-XH CONNECTORS"
- note added: "WS-90 CONNECTOR TO CONNECT TO THE MAIN BOARD"
- note added: "WS-90 CONNECTOR TO CONNECT TO THE RADIO BOARD"
- note added: "WS-90 CONNECTORS"
- note removed: "CONNECTORS"
- moved on the sheet: C37, C38, C39, C40, C41, C44, C56, C57, D3, D4, D5, D6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

Commit message: changed buck converters
Parts:
- removed C10, C24: 1u, symbol Device:C
- removed C11, C15, C16, C25, C28, C29: 100n, symbol Device:C
- removed C13, C14, C17, C18, C19, C20, C21, C26, C27, C30, C31, C32, C33, C34: 22u, symbol Device:C
- removed C22, C35: 100p, symbol Device:C
- removed C23, C36: 22n, symbol Device:C
- removed L1, L2: 2.2uH, symbol Device:L_Iron
- removed R12, R26: 0, symbol Device:R
- removed R18, R29: 470k, symbol Device:R
- removed R19: 220K, symbol Device:R
- removed R20, R31: 150k, symbol Device:R
- removed R21, R32: 330k, symbol Device:R
- removed R22, R33: 30K, symbol Device:R
- removed R24, R36: 5.1K, symbol Device:R
- removed R25, R38: 100K, symbol Device:R
- removed R30: 160K, symbol Device:R
- removed SW1: SW_SPST, symbol Switch:SW_SPST
- removed TP11, TP7: TestPoint, symbol Connector:TestPoint
- removed U10, U12: TPS568230RJER, symbol TPS568230RJER:TPS568230RJER
- added C100, C105: 10nF, symbol Device:C
- added C101, C108: 12uF, symbol Device:C
- added C102, C109: 3.9nF, symbol Device:C
- added C103, C107: 0.1uF, symbol Device:C
- added C104, C106: 10uF/25V, symbol Device:C_Polarized
- added L8, L9: 10uH, symbol Device:L
- added R74: 30.9K, symbol Device:R
- added R75, R80: 10K, symbol Device:R
- added R76: 6.8K, symbol Device:R
- added R77, R78: 100K, symbol Device:R
- added R79: 44.2K, symbol Device:R
- added R81: 6,8K, symbol Device:R
- added U27, U28: MP2307, MP2307:SO-8_EP, symbol MP2307:MP2307
Connections:
- net 3V8_OUT: now also C101.1, L8.2, R74.1
- net 5V_OUT: now also C108.1, L9.2, R79.1
- net GND: now also C101.2, C103.1, C104.2, C106.2, C107.1, C108.2, R75.2, R76.1, R80.2, R81.1, U27.4 (4_GND), U28.4 (4_GND)
- net VBAT: now also C104.1, C106.1, R77.2, R78.2, U27.2 (2_IN), U28.2 (2_IN)
- new net: R78.1, U28.7 (7_EN)
- new net: C102.1, R76.2
- new net: C100.2, L8.1, U27.3 (3_SW)
- new net: C109.1, R81.2
- new net: C109.2, U28.6 (6_COMP)
- new net: C105.1, U28.1 (1_BS)
- new net: C105.2, L9.1, U28.3 (3_SW)
- new net: R79.2, R80.1, U28.5 (5_FB)
- new net: C107.2, U28.8 (8_SS)
- new net: C100.1, U27.1 (1_BS)
- new net: R74.2, R75.1, U27.5 (5_FB)
- new net: C102.2, U27.6 (6_COMP)
- new net: R77.1, U27.7 (7_EN)
- new net: C103.2, U27.8 (8_SS)
Other:
- note added: "3V8@4A PEAK CHANNEL - 1"
- note added: "5V@4A PEAK CHANNEL - 1"
- note added: "VOUT = 10.81 X (VOUT - 0.925) (K ohms)"
- note removed: "4.2V@8A PEAK CHANNEL - 2"
- note removed: "5V@8A PEAK CHANNEL - 1"
- moved on the sheet: C42, C43, C45, C46, C47, C48, C49, C50, C51, C52, C53, C54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

Commit message: migrating kicad 9 to 10
Parts:
- removed BT9: Battery_Cell, symbol Device:Battery_Cell
- removed C37: 100nf, symbol Device:C_Small
- removed C38, C39: 22uF, symbol Device:C
- removed C40, C41, C44: 1u, symbol Device:C_Small
- removed C56: 100n, symbol Device:C_Small
- removed C57: 100 nF, symbol Device:C_Small
- removed D3, D4, D7: LED, symbol Device:LED
- removed IP2: ~, symbol IP2368:IP2368
- removed J18: USB_C_Receptacle_USB2.0_16P, symbol Connector:USB_C_Receptacle_USB2.0_16P
- removed L4: 10uH, symbol Device:L
- removed Q1, Q2, Q3, Q4, Q5, Q6, Q7, Q8, Q9: NMOS, symbol Simulation_SPICE:NMOS
- removed R17: 10k, symbol Device:R_Small
- removed R28, R34: 1K, symbol Device:R
- removed R37: 10k, symbol Device:R
- removed R39: 12.4K, symbol Device:R
- removed R40: 6.2k, symbol Device:R
- removed R42, R43: 5m, symbol Device:R
- removed U28: MP2307, MP2307:SO-8_EP, symbol MP2307:MP2307
- added BT2: 18650, Battery:BatteryHolder_Keystone_1042_1x18650, symbol Device:Battery_Cell
- added C20, C22: 470uF, Capacitor_SMD:CP_Elec_10x10, symbol Device:C_Polarized
- added C21, C31: 100 nF, Capacitor_SMD:C_1206_3216Metric_Pad1.33x1.80mm_HandSolder, symbol Device:C
- added C29: 470pF, Capacitor_SMD:C_1206_3216Metric_Pad1.33x1.80mm_HandSolder, symbol Device:C
- added C30: 220nF, Capacitor_SMD:C_1206_3216Metric_Pad1.33x1.80mm_HandSolder, symbol Device:C
- added D1, D2, D4: SK54, Diode_SMD:D_SMC_Handsoldering, symbol Device:D
- added D3: SMAJ22A, Diode_SMD:D_SMA_Handsoldering, symbol Diode:SMAJ22A
- added D7: D, Diode_SMD:D_SMC_Handsoldering, symbol Device:D
- added J10: Barrel_Jack_Switch, Connector_BarrelJack:BarrelJack_Horizontal, symbol Connector:Barrel_Jack_Switch
- added L2: 10uH, Inductor_SMD:L_10.4x10.4_H4.8, symbol Device:L
- added Q1, Q4: Q_NMOS_GSD, Package_TO_SOT_SMD:SOT-23, symbol Transistor_FET:Q_NMOS_GSD
- added Q2, Q3: Q_NMOS_SGD, Package_SO:SOIC-8_3.9x4.9mm_P1.27mm, symbol Transistor_FET:Q_NMOS_SGD
- added Q5, Q6: Q_PMOS_SGD, Package_SO:SOIC-8_3.9x4.9mm_P1.27mm, symbol Transistor_FET:Q_PMOS_SGD
- added R22: 0.05Ω, Resistor_SMD:R_2512_6332Metric, symbol Device:R
- added R25: 4.7k, Resistor_SMD:R_0805_2012Metric_Pad1.20x1.40mm_HandSolder, symbol Device:R
- added R30: 120, Resistor_SMD:R_0805_2012Metric_Pad1.20x1.40mm_HandSolder, symbol Device:R
- added R32: 0, Resistor_SMD:R_0805_2012Metric_Pad1.20x1.40mm_HandSolder, symbol Device:R
- added R36: 10k, Resistor_SMD:R_0805_2012Metric_Pad1.20x1.40mm_HandSolder, symbol Device:R_Small
- added U7: MP2307, Package_SO:SOIC-8-1EP_3.9x4.9mm_P1.27mm_EP2.29x3mm_ThermalVias, symbol MP2307:MP2307
- added U8: CN3702, Package_SO:TSSOP-16_4.4x5mm_P0.65mm, symbol CN3702:CN3702
- BT1: renamed from BT2; value Battery_Cell -> 18650; footprint (none) -> Battery:BatteryHolder_Keystone_1042_1x18650
- BT3, BT4, BT5, BT6, BT7, BT8: value Battery_Cell -> 18650; footprint (none) -> Battery:BatteryHolder_Keystone_1042_1x18650
- C1: renamed from C6; footprint (none) -> Capacitor_SMD:C_1206_3216Metric_Pad1.33x1.80mm_HandSolder
- C10: renamed from C47; footprint (none) -> Capacitor_SMD:C_1206_3216Metric_Pad1.33x1.80mm_HandSolder
- C11: renamed from C48; footprint (none) -> Capacitor_SMD:C_1206_3216Metric_Pad1.33x1.80mm_HandSolder
- C12: renamed from C49; footprint (none) -> Capacitor_SMD:C_1206_3216Metric_Pad1.33x1.80mm_HandSolder
- C13: renamed from C50; footprint (none) -> Capacitor_SMD:C_1206_3216Metric_Pad1.33x1.80mm_HandSolder
- C14: renamed from C51; footprint (none) -> Capacitor_SMD:C_1206_3216Metric_Pad1.33x1.80mm_HandSolder
- C15: renamed from C52; footprint (none) -> Capacitor_SMD:C_1206_3216Metric_Pad1.33x1.80mm_HandSolder
- C16: renamed from C53; footprint (none) -> Capacitor_SMD:C_1206_3216Metric_Pad1.33x1.80mm_HandSolder
- C17: renamed from C54; footprint (none) -> Capacitor_SMD:C_1206_3216Metric_Pad1.33x1.80mm_HandSolder
- C18: renamed from C55; footprint (none) -> Capacitor_SMD:C_1206_3216Metric_Pad1.33x1.80mm_HandSolder
- C19: renamed from C100; footprint (none) -> Capacitor_SMD:C_1206_3216Metric_Pad1.33x1.80mm_HandSolder
- C2: renamed from C7; footprint (none) -> Capacitor_SMD:C_1206_3216Metric_Pad1.33x1.80mm_HandSolder
- C23: renamed from C104; footprint (none) -> CP_Elec_10x10
- C24: renamed from C103; footprint (none) -> Capacitor_SMD:C_1206_3216Metric_Pad1.33x1.80mm_HandSolder
- C25: renamed from C101; footprint (none) -> Capacitor_SMD:C_1206_3216Metric_Pad1.33x1.80mm_HandSolder
- C26: renamed from C102; footprint (none) -> Capacitor_SMD:C_1206_3216Metric_Pad1.33x1.80mm_HandSolder
- C27: renamed from C105; footprint (none) -> Capacitor_SMD:C_1206_3216Metric_Pad1.33x1.80mm_HandSolder
- C28: renamed from C106; footprint (none) -> Capacitor_SMD:C_1206_3216Metric_Pad1.33x1.80mm_HandSolder
- C3: renamed from C8; footprint (none) -> Capacitor_SMD:C_1206_3216Metric_Pad1.33x1.80mm_HandSolder
- C32: renamed from C107; footprint (none) -> Capacitor_SMD:C_1206_3216Metric_Pad1.33x1.80mm_HandSolder
- C33: renamed from C108; footprint (none) -> Capacitor_SMD:C_1206_3216Metric_Pad1.33x1.80mm_HandSolder
- C34: renamed from C109; footprint (none) -> Capacitor_SMD:C_1206_3216Metric_Pad1.33x1.80mm_HandSolder
- C4: renamed from C9; footprint (none) -> Capacitor_SMD:C_1206_3216Metric_Pad1.33x1.80mm_HandSolder
- C5: renamed from C42; footprint (none) -> Capacitor_SMD:C_1206_3216Metric_Pad1.33x1.80mm_HandSolder
- C6: renamed from C43; footprint (none) -> Capacitor_SMD:C_1206_3216Metric_Pad1.33x1.80mm_HandSolder
- C7: renamed from C12; footprint (none) -> Capacitor_SMD:C_1206_3216Metric_Pad1.33x1.80mm_HandSolder
- C8: renamed from C45; footprint (none) -> Capacitor_SMD:C_1206_3216Metric_Pad1.33x1.80mm_HandSolder
- C9: renamed from C46; footprint (none) -> Capacitor_SMD:C_1206_3216Metric_Pad1.33x1.80mm_HandSolder
- D5, D6: footprint (none) -> LED_SMD:LED_0805_2012Metric_Pad1.15x1.40mm_HandSolder
- F1: footprint (none) -> Fuse:Fuse_2920_7451Metric_Pad2.10x5.45mm_HandSolder
- J1: renamed from J14; footprint (none) -> Connector_JST:JST_VH_B2P-VH-B_1x02_P3.96mm_Vertical
- J2: renamed from J15; footprint (none) -> Connector_JST:JST_VH_B2P-VH-B_1x02_P3.96mm_Vertical
- J3: renamed from J16; footprint (none) -> Connector_JST:JST_VH_B2P-VH-B_1x02_P3.96mm_Vertical
- J4: renamed from J3; footprint (none) -> Connector_JST:JST_VH_B2P-VH-B_1x02_P3.96mm_Vertical
- J5: renamed from J4; footprint (none) -> Connector_JST:JST_VH_B2P-VH-B_1x02_P3.96mm_Vertical
- J6: footprint (none) -> Connector_JST:JST_XH_B2B-XH-A_1x02_P2.50mm_Vertical
- J7: renamed from J8; footprint (none) -> Connector_JST:JST_XH_B2B-XH-A_1x02_P2.50mm_Vertical
- J8: renamed from J17; footprint (none) -> Connector_JST:JST_XH_B3B-XH-A_1x03_P2.50mm_Vertical
- J9: renamed from J58; footprint (none) -> Connector_JST:JST_XH_B3B-XH-A_1x03_P2.50mm_Vertical
- L1: renamed from L3; value 1.5uH -> 2.2uH; footprint (none) -> Inductor_SMD:L_7.3x7.3_H3.5
- L3: renamed from L8; footprint (none) -> Inductor_SMD:L_10.4x10.4_H4.8
- L4: renamed from L9; footprint (none) -> Inductor_SMD:L_10.4x10.4_H4.8
- R1: renamed from R5; footprint (none) -> Resistor_SMD:R_1206_3216Metric_Pad1.30x1.75mm_HandSolder
- R10: renamed from R44; footprint (none) -> Resistor_SMD:R_0805_2012Metric_Pad1.20x1.40mm_HandSolder
- R11: renamed from R45; footprint (none) -> Resistor_SMD:R_0805_2012Metric_Pad1.20x1.40mm_HandSolder
- R12: renamed from R14; footprint (none) -> Resistor_SMD:R_0805_2012Metric_Pad1.20x1.40mm_HandSolder
- R13: renamed from R15; footprint (none) -> Resistor_SMD:R_0805_2012Metric_Pad1.20x1.40mm_HandSolder
- R14: renamed from R16; footprint (none) -> Resistor_SMD:R_0805_2012Metric_Pad1.20x1.40mm_HandSolder
- R15: renamed from R46; footprint (none) -> Resistor_SMD:R_0805_2012Metric_Pad1.20x1.40mm_HandSolder
- R17: renamed from R47; footprint (none) -> Resistor_SMD:R_0805_2012Metric_Pad1.20x1.40mm_HandSolder
- R18: renamed from R48; footprint (none) -> Resistor_SMD:R_0805_2012Metric_Pad1.20x1.40mm_HandSolder
- R19: renamed from R49; footprint (none) -> Resistor_SMD:R_0805_2012Metric_Pad1.20x1.40mm_HandSolder
- R2: renamed from R6; footprint (none) -> Resistor_SMD:R_0805_2012Metric_Pad1.20x1.40mm_HandSolder
- R20: renamed from R23; footprint (none) -> Resistor_SMD:R_Shunt_Vishay_WSK2512_6332Metric_T2.21mm
- R21: renamed from R50; footprint (none) -> Resistor_SMD:R_0805_2012Metric_Pad1.20x1.40mm_HandSolder
- R23: renamed from R77; footprint (none) -> Resistor_SMD:R_0805_2012Metric_Pad1.20x1.40mm_HandSolder
- R24: renamed from R74; footprint (none) -> Resistor_SMD:R_0805_2012Metric_Pad1.20x1.40mm_HandSolder
- R26: renamed from R75; footprint (none) -> Resistor_SMD:R_0805_2012Metric_Pad1.20x1.40mm_HandSolder
- R27: value 1K -> 4.7k; footprint (none) -> Resistor_SMD:R_0805_2012Metric_Pad1.20x1.40mm_HandSolder
- R28: renamed from R76; footprint (none) -> Resistor_SMD:R_0805_2012Metric_Pad1.20x1.40mm_HandSolder
- R29: renamed from R78; footprint (none) -> Resistor_SMD:R_0805_2012Metric_Pad1.20x1.40mm_HandSolder
- R3: renamed from R7; footprint (none) -> Resistor_SMD:R_0805_2012Metric_Pad1.20x1.40mm_HandSolder
- R31: renamed from R79; value 44.2K -> 26.1K; footprint (none) -> Resistor_SMD:R_0805_2012Metric_Pad1.20x1.40mm_HandSolder
- R33: renamed from R80; footprint (none) -> Resistor_SMD:R_0805_2012Metric_Pad1.20x1.40mm_HandSolder
- R34: renamed from R81; footprint (none) -> Resistor_SMD:R_0805_2012Metric_Pad1.20x1.40mm_HandSolder
- R35: value 27K -> 100k; footprint (none) -> Resistor_SMD:R_0805_2012Metric_Pad1.20x1.40mm_HandSolder
- R4: renamed from R8; footprint (none) -> Resistor_SMD:R_0805_2012Metric_Pad1.20x1.40mm_HandSolder
- R5: renamed from R9; footprint (none) -> Resistor_SMD:R_0805_2012Metric_Pad1.20x1.40mm_HandSolder
- R6: renamed from R10; footprint (none) -> Resistor_SMD:R_1206_3216Metric_Pad1.30x1.75mm_HandSolder
- R7: renamed from R11; footprint (none) -> Resistor_SMD:R_0805_2012Metric_Pad1.20x1.40mm_HandSolder
- R8: renamed from R41; footprint (none) -> Resistor_SMD:R_0805_2012Metric_Pad1.20x1.40mm_HandSolder
- R9: renamed from R13; footprint (none) -> Resistor_SMD:R_0805_2012Metric_Pad1.20x1.40mm_HandSolder
- TH1: footprint (none) -> Connector_PinHeader_2.54mm:PinHeader_1x02_P2.54mm_Vertical
- TP1: renamed from TP3; footprint (none) -> TestPoint:TestPoint_Pad_D1.0mm
- TP2: renamed from TP4; footprint (none) -> TestPoint:TestPoint_Pad_D1.0mm
- TP3: renamed from TP5; footprint (none) -> TestPoint:TestPoint_Pad_D1.0mm
- TP4: renamed from TP6; footprint (none) -> TestPoint:TestPoint_Pad_D1.0mm
- TP5: renamed from TP12; footprint (none) -> TestPoint:TestPoint_Pad_D1.0mm
- TP6: renamed from TP8; footprint (none) -> TestPoint:TestPoint_Pad_D1.0mm
- TP7: renamed from TP9; footprint (none) -> TestPoint:TestPoint_Pad_D1.0mm
- TP8: renamed from TP10; footprint (none) -> TestPoint:TestPoint_Pad_D1.0mm
- U1: renamed from U7; footprint (none) -> Package_TO_SOT_SMD:SOT-23-6_Handsoldering
- U2: renamed from U26; footprint (none) -> Package_TO_SOT_SMD:SOT-23-6_Handsoldering
- U3: renamed from U9; footprint (none) -> Package_TO_SOT_SMD:SOT-23-6_Handsoldering
- U4: renamed from U13; footprint (none) -> Package_DFN_QFN:VQFN-20-1EP_3x3mm_P0.45mm_EP1.55x1.55mm_ThermalVias
- U6: renamed from U27; footprint MP2307:SO-8_EP -> Package_SO:SOIC-8-1EP_3.9x4.9mm_P1.27mm_EP2.29x3mm_ThermalVias
- renumbered U11 to U5
Connections:
- net VCC-3 is gone; now on net VCC: C5.2, R21.2, U4.17 (VCC)
- net 3V3_OUT: now also C33.1, L4.2, R31.1, R36.1; no longer C11.1, C12.1, C13.1, C14.1, C15.1, C16.1, C17.1, L1.2, R11.1, TP5.1
- net 5V_OUT: now also C11.1, C12.1, C13.1, C14.1, C15.1, C16.1, C17.1, L1.2, R11.1, TP5.1; no longer C33.1, L4.2, R31.1
- net BAT+: now also C22.1, Q6.1 (S), Q6.2 (SOURCE), Q6.3 (SOURCE), R22.2, U8.14 (BAT)
- net BAT-: now also BT5.2 (-), Q1.2 (S), Q2.1 (S), Q2.2 (SOURCE), Q2.3 (SOURCE)
- net BAT_MID: now also BT5.1 (+), BT2.2 (-), Q4.2 (S); no longer BT5.2 (-)
- net GND: now also R35.1, U6.9 (4_GND), C20.2, C22.2, C29.2, C30.2, C31.2, D3.2 (A2), D4.2 (A), J10.2, J10.3, Q3.1 (S), Q3.2 (SOURCE), Q3.3 (SOURCE), R32.2, U7.4 (4_GND), U7.9 (4_GND), U8.10 (TEST), U8.2 (PGND), U8.3 (GND); no longer D5.1 (K), D6.2 (A), R35.2
- net VBAT: now also D7.1 (K), Q6.5 (D), Q6.6 (DRAIN), Q6.7 (DRAIN), Q6.8 (DRAIN), U7.2 (2_IN)
- net at R29.1: now also U7.7 (7_EN)
- net at TH1.1: now also U8.6 (TEMP)
- net at R27.2: now also D6.2 (A)
- net at U1.6 (OUT): now also Q4.1 (G)
- net at C34.2: now also U7.6 (6_COMP)
- net at C27.1: now also U7.1 (1_BS)
- net at C27.2, L4.1: now also U7.3 (3_SW)
- net at R31.2, R33.1: now also U7.5 (5_FB)
- net at C32.2: now also U7.8 (8_SS)
- net at BT1.1 (+), BT3.1 (+), BT4.1 (+)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: now also BT2.1 (+); no longer BT5.1 (+)
- net SDA: now reaches J8.1 (Pin_1), R14.1, TP6.1, U5.4 (SDA)
- net SDA: no longer J8.3 (Pin_3), U5.3 (~{Alert})
- net SCL: now reaches J8.2 (Pin_2), R13.1, TP7.1, U5.5 (SCL)
- net at R6.1: now also Q1.3 (D)
- net at U3.6 (OUT): now also Q1.1 (G)
- net at U2.1 (OD): now also Q2.4 (G)
- net at U2.2 (OC): now also Q3.4 (G)
- net at D6.1 (K): now also U8.5 (DONE); no longer D5.2 (A)
- net at R1.1: now also Q4.3 (D)
- net 12V: now reaches R27.1
- net 12V: now also R35.2, C20.1, C21.1, D1.1 (K), D7.2 (A), Q5.5 (D), Q5.6 (DRAIN), Q5.7 (DRAIN), Q5.8 (DRAIN), Q6.4 (G), R25.1, U8.15 (VCC)
- new net: C31.1, U8.11 (COM3)
- new net: L2.2, R22.1, U8.13 (CSP)
- new net: R30.1, U8.9 (COM2)
- new net: C30.1, R30.2
- new net: D1.2 (A), D3.1 (A1), J10.1
- new net: Q2.5 (D), Q2.6 (DRAIN), Q2.7 (DRAIN), Q2.8 (DRAIN), Q3.5 (D), Q3.6 (DRAIN), Q3.7 (DRAIN), Q3.8 (DRAIN)
- new net: D2.1 (K), D4.1 (K), L2.1
- new net: C21.2, U8.1 (VG)
- new net: R32.1, U8.7 (EOC)
- new net: D5.1 (K), U8.4 (CHRG)
- new net: D5.2 (A), R25.2
- new net: Q5.4 (G), U8.16 (DRV)
- new net: C29.1, U8.8 (COM1)
- new net: D2.2 (A), Q5.1 (S), Q5.2 (SOURCE), Q5.3 (SOURCE)
- new net GPIO: J8.3 (Pin_3), R36.2, U5.3 (~{Alert})
- no-connect marks 13 -> 6
Other:
- note added: "3V3@4A PEAK CHANNEL - 1"
- note added: "5V@8A PEAK CHANNEL - 1"
- note added: "INPUT 12V@65W"
- note added: "JST-VH CONNECTOR TO CONNECT TO THE MAIN BOARD"
- note added: "JST-VH CONNECTOR TO CONNECT TO THE RADIO BOARD"
- note added: "JST-VH CONNECTORS"
- note added: "POWER INPUT"
- note removed: "10K"
- note removed: "3V3@8A PEAK CHANNEL - 1"
- note removed: "5V@4A PEAK CHANNEL - 1"
- note removed: "R42- 6.2K , CONFIGURE IT FOR 2S R32 - 10K, SETS MAX CHARGE VOLTAGE AS 4.2V FOR 1 CELL, 8.4V TOTAL R44 - 27K , SETS THE PD INPUT POWER LIMIT TO 100W R43 - 12.4K, TELLS THAT THE TOTAL CURRENT OF 4P CELLS ARE 10,000 mAh"
- note removed: "TYPE-C CHARGER"
- note removed: "WS-90 CONNECTOR TO CONNECT TO THE MAIN BOARD"
- note removed: "WS-90 CONNECTOR TO CONNECT TO THE RADIO BOARD"
- note removed: "WS-90 CONNECTORS"
