File: kicad/power-supply/power-supply.kicad_sch (KiCad schematic)
At the start: 122 parts, among them J1 Conn_01x02, J10 Barrel_Jack_Switch, J2 Conn_01x02, J3 Conn_01x02, J4 Conn_01x02, J5 Conn_01x02, J6 Conn_01x02, J7 Conn_01x02, J8 Conn_01x03, J9 Conn_01x03, Q1 Q_NMOS_GSD, Q2 Q_NMOS_SGD, Q3 Q_NMOS_SGD, Q4 Q_NMOS_GSD, Q5 Q_PMOS_SGD, Q6 Q_PMOS_SGD, U1 HY2213-BB3A, U2 HY2120, U3 HY2213-BB3A, U4 TPS568230RJER, U5 INA226, U6 MP2307, U7 MP2307, U8 CN3702

Commit message: upddate
Parts:
- removed C22: 470uF, Capacitor_SMD:CP_Elec_10x10, symbol Device:C_Polarized
- removed C29: 470pF, Capacitor_SMD:C_1206_3216Metric_Pad1.33x1.80mm_HandSolder, symbol Device:C
- removed C30: 220nF, Capacitor_SMD:C_1206_3216Metric_Pad1.33x1.80mm_HandSolder, symbol Device:C
- removed C31: 100 nF, Capacitor_SMD:C_1206_3216Metric_Pad1.33x1.80mm_HandSolder, symbol Device:C
- removed D1, D2, D4: SK54, Diode_SMD:D_SMC_Handsoldering, symbol Device:D
- removed D3: SMAJ22A, Diode_SMD:D_SMA_Handsoldering, symbol Diode:SMAJ22A
- removed D5, D6: LED, LED_SMD:LED_0805_2012Metric_Pad1.15x1.40mm_HandSolder, symbol Device:LED
- removed D7: D, Diode_SMD:D_SMC_Handsoldering, symbol Device:D
- removed J10: Barrel_Jack_Switch, Connector_BarrelJack:BarrelJack_Horizontal, symbol Connector:Barrel_Jack_Switch
- removed Q5, Q6: Q_PMOS_SGD, Package_SO:SOIC-8_3.9x4.9mm_P1.27mm, symbol Transistor_FET:Q_PMOS_SGD
- removed R22: 0.05Ω, Resistor_SMD:R_2512_6332Metric, symbol Device:R
- removed R35: 100k, Resistor_SMD:R_0805_2012Metric_Pad1.20x1.40mm_HandSolder, symbol Device:R
- removed TH1: Thermistor_NTC, Connector_PinHeader_2.54mm:PinHeader_1x02_P2.54mm_Vertical, symbol Device:Thermistor_NTC
- removed U8: CN3702, Package_SO:TSSOP-16_4.4x5mm_P0.65mm, symbol CN3702:CN3702
- added C18: 2.2uF, symbol Device:C
- added C19, C27: 1uF, symbol Device:C
- added C22, C23: 100nF, symbol Device:C
- added C24, C25: 10uF, symbol Device:C
- added C26: 22pF, symbol Device:C
- added D100: SK54, Diode_SMD:D_SMC_Handsoldering, symbol Device:D
- added D101, D102: LED, symbol Device:LED
- added D103: BAT54W, Package_TO_SOT_SMD:SOT-323_SC-70, symbol Diode:BAT54W
- added D99: SMAJ22A, Diode_SMD:D_SMA_Handsoldering, symbol Diode:SMAJ22A
- added J18: Barrel_Jack_Switch, Connector_BarrelJack:BarrelJack_Horizontal, symbol Connector:Barrel_Jack_Switch
- added Q1, Q2: NMOS, symbol Simulation_SPICE:NMOS
- added R17: 10m (0.01), symbol Device:R
- added R26: 4.7K, symbol Device:R
- added R28: 10, symbol Device:R
- added R29: 300K, symbol Device:R
- added R31: R, symbol Device:R
- added R33: 82K, symbol Device:R
- added R34: 10K, symbol Device:R
- added U28: BQ24650RVAR, BQ24650RVAR:QFN50P350X350X100-17N, symbol BQ24650RVAR:BQ24650RVAR
- C21: value 100 nF -> 1uF; footprint Capacitor_SMD:C_1206_3216Metric_Pad1.33x1.80mm_HandSolder -> (none)
- L2: value 10uH -> 6.8uH; footprint Inductor_SMD:L_10.4x10.4_H4.8 -> (none)
- R25: value 4.7k -> 4.7K; footprint Resistor_SMD:R_0805_2012Metric_Pad1.20x1.40mm_HandSolder -> (none)
- R27: value 4.7k -> 2; footprint Resistor_SMD:R_0805_2012Metric_Pad1.20x1.40mm_HandSolder -> (none)
- R30: value 120 -> 100K; footprint Resistor_SMD:R_0805_2012Metric_Pad1.20x1.40mm_HandSolder -> (none)
- R32: value 0 -> R; footprint Resistor_SMD:R_0805_2012Metric_Pad1.20x1.40mm_HandSolder -> (none)
- renumbered BT1 to BT2, BT8 to BT?, BT7 to BT?, BT3 to BT?, BT4 to BT?, BT6 to BT?, BT2 to BT?, BT5 to BT?, C19 to C100, C25 to C101, C26 to C102, C24 to C103, C23 to C104, C27 to C105, C28 to C106, C32 to C107, C33 to C108, C34 to C109, C7 to C12, C5 to C42, C6 to C43, C8 to C45, C9 to C46, C10 to C47, C11 to C48, C12 to C49, C13 to C50, C14 to C51, C15 to C52, C16 to C53, C17 to C54, C18 to C55, C1 to C6, C2 to C7, C3 to C8, C4 to C9, J1 to J14, J2 to J15, J3 to J16, J8 to J17, J4 to J3, J5 to J4, J9 to J58, J7 to J8, L1 to L3, L3 to L8, L4 to L9, Q2 to Q?, Q3 to Q?, Q1 to Q?, Q4 to Q?, R6 to R10, R7 to R11, R9 to R13, R12 to R14, R13 to R15, R14 to R16, R20 to R23, R8 to R41, R10 to R44, R11 to R45, R15 to R46, R17 to R47, R18 to R48, R19 to R49, R1 to R5, R21 to R50, R2 to R6, R3 to R7, R24 to R74, R26 to R75, R28 to R76, R23 to R77, R29 to R78, R31 to R79, R4 to R8, R33 to R80, R34 to R81, R5 to R9, TP8 to TP10, TP5 to TP12, TP1 to TP3, TP2 to TP4, TP3 to TP5, TP4 to TP6, TP6 to TP8, TP7 to TP9, U5 to U11, U4 to U13, U2 to U26, U6 to U27, U1 to U7, U3 to U9, U7 to U?
Connections:
- net 12V: now also D100.1 (K), Q1.1 (D), R26.2, R28.1, R31.1; no longer C21.1, R27.1
- net GND: now also C21.2, R30.2, C18.2, C19.2, C24.2, C25.2, C27.2, D99.2 (A2), J18.2, J18.3, Q2.3 (S), R34.2, U28.11 (GND), U28.17 (EP)
- net at R27.2: now also C18.1
- net SRP: now reaches L2.2
- net SRP: now also C23.1, R17.1, U28.10 (SRP)
- net at R30.1: now also C26.2, R29.2, U28.8 (VFB)
- net at L2.1: now also C22.2, Q1.3 (S), Q2.1 (D), U28.14 (PH)
- net at R32.1: now also R31.2, R33.2, R34.1, U28.2 (MPPSET), U28.4 (TS)
- net at R25.2: now also D101.2 (A)
- new net: D100.2 (A), D99.1 (A1), J18.1, R27.1
- new net: C19.1, R28.2, U28.1 (VCC)
- new net: D102.1 (K), U28.5 (STAT2)
- new net: D102.2 (A), R26.1
- new net: C23.2, C24.1, C25.1, C26.1, R17.2, R29.1, U28.9 (SRN)
- new net: Q2.2 (G), U28.13 (LODRV)
- new net: C27.1, R33.1, U28.6 (VREF), U28.7 (TERM_EN)
- new net: C22.1, D103.3 (K), U28.16 (BTST)
- new net: C21.1, D103.1 (A), U28.12 (REGN)
- new net: D101.1 (K), U28.3 (STAT1)
- new net: Q1.2 (G), U28.15 (HIDRV)
Other:
- note added: "BATTERY CHARGER"
