File: kicad/GPIO-board/GPIO-board.kicad_sch (KiCad schematic)
At the start: 25 parts, among them J1 BANANA JACK LV, J2 BANANA JACK HV, U1 MP2307

Commit message: made overall schematic
Parts:
- added J3: Conn_02x15_Top_Bottom, symbol Connector_Generic:Conn_02x15_Top_Bottom
- added J4: Conn_01x04_Pin, symbol Connector:Conn_01x04_Pin
Connections:
- net GND: now also A1.13 (GND), A1.18 (GND), A1.23 (GND), A1.28 (GND), A1.3 (GND), A1.33 (AGND), A1.38 (GND), A1.8 (GND), A1.D2 (GND), A1.TP1 (USB_GND), J3.29 (Pin_29), J3.30 (Pin_30), J4.2 (Pin_2)
- net P0: now reaches A1.1 (GPIO0)
- net P0: now also J3.1 (Pin_1)
- net P7: now reaches A1.10 (GPIO7)
- net P7: now also J3.8 (Pin_8)
- net P8: now reaches A1.11 (GPIO8)
- net P8: now also J3.9 (Pin_9)
- net P9: now reaches A1.12 (GPIO9)
- net P9: now also J3.10 (Pin_10)
- net P10: now reaches A1.14 (GPIO10)
- net P10: now also J3.11 (Pin_11)
- net P11: now reaches A1.15 (GPIO11)
- net P11: now also J3.12 (Pin_12)
- net P12: now reaches A1.16 (GPIO12)
- net P12: now also J3.13 (Pin_13)
- net P13: now reaches A1.17 (GPIO13)
- net P13: now also J3.14 (Pin_14)
- net P14: now reaches A1.19 (GPIO14)
- net P14: now also J3.15 (Pin_15)
- net P1: now reaches A1.2 (GPIO1)
- net P1: now also J3.2 (Pin_2)
- net P15: now reaches A1.20 (GPIO15)
- net P15: now also J3.16 (Pin_16)
- net P16: now reaches A1.21 (GPIO16)
- net P16: now also J3.17 (Pin_17)
- net P17: now reaches A1.22 (GPIO17)
- net P17: now also J3.18 (Pin_18)
- net P18: now reaches A1.24 (GPIO18)
- net P18: now also J3.19 (Pin_19)
- net P19: now reaches A1.25 (GPIO19)
- net P19: now also J3.20 (Pin_20)
- net P20: now reaches A1.26 (GPIO20)
- net P20: now also J3.21 (Pin_21)
- net P21: now reaches A1.27 (GPIO21)
- net P21: now also J3.22 (Pin_22)
- net P22: now reaches A1.29 (GPIO22)
- net P22: now also J3.23 (Pin_23)
- net P26: now reaches A1.31 (GPIO26_ADC0)
- net P26: now also J3.24 (Pin_24)
- net P27: now reaches A1.32 (GPIO27_ADC1)
- net P27: now also J3.25 (Pin_25)
- net P28: now reaches A1.34 (GPIO28_ADC2)
- net P28: now also J3.26 (Pin_26)
- net ADC_VREF: now reaches A1.35 (ADC_VREF)
- net ADC_VREF: now also J3.27 (Pin_27)
- net +3V3: now reaches A1.36 (3V3)
- net +3V3: now also J3.28 (Pin_28), J4.1 (Pin_1)
- net P2: now reaches A1.4 (GPIO2)
- net P2: now also J3.3 (Pin_3)
- net P3: now reaches A1.5 (GPIO3)
- net P3: now also J3.4 (Pin_4)
- net P4: now reaches A1.6 (GPIO4)
- net P4: now also J3.5 (Pin_5)
- net P5: now reaches A1.7 (GPIO5)
- net P5: now also J3.6 (Pin_6)
- net P6: now reaches A1.9 (GPIO6)
- net P6: now also J3.7 (Pin_7)
- net USB_DM: now reaches A1.TP2 (USB_DM)
- net USB_DM: now also J4.3 (Pin_3)
- net USB_DP: now reaches A1.TP3 (USB_DP)
- net USB_DP: now also J4.4 (Pin_4)
- no-connect marks 0 -> 5
Other:
- moved on the sheet: A1

Commit message: worke don the usb hub
Parts:
- renumbered RV to RV2
Changed lines of the file:
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@@
 		(dnp no)
 		(fields_autoplaced yes)
-		(property "Reference" "#PWR05"
+		(property "Reference" "#PWR0104"
 			(at 130.81 86.36 0)
 			(effects
@@
 			(project "OVERALL"
 				(path "/0e81c85d-86ab-4d5d-8c59-60b8e6f89475/0d6bced7-1bbd-4604-8bae-89d93aa4735e"
-					(reference "#PWR05")
+					(reference "#PWR0104")
 					(unit 1)
 				)
@@
 		(dnp no)
 		(fields_autoplaced yes)
-		(property "Reference" "#PWR03"
+		(property "Reference" "#PWR0103"
 			(at 269.24 63.5 0)
 			(effects
@@
 			(project "OVERALL"
 				(path "/0e81c85d-86ab-4d5d-8c59-60b8e6f89475/0d6bced7-1bbd-4604-8bae-89d93aa4735e"
-					(reference "#PWR03")
+					(reference "#PWR0103")
 					(unit 1)
 				)
@@
 		(dnp no)
 		(fields_autoplaced yes)
-		(property "Reference" "#PWR01"
+		(property "Reference" "#PWR0109"
 			(at 152.4 62.23 0)
 			(effects
@@
 			(project "OVERALL"
 				(path "/0e81c85d-86ab-4d5d-8c59-60b8e6f89475/0d6bced7-1bbd-4604-8bae-89d93aa4735e"
-					(reference "#PWR01")
+					(reference "#PWR0109")
 					(unit 1)
 				)
@@
 		(dnp no)
 		(fields_autoplaced yes)
-		(property "Reference" "#PWR02"
+		(property "Reference" "#PWR0102"
 			(at 148.59 118.11 0)
 			(effects
@@
 			(project "OVERALL"
 				(path "/0e81c85d-86ab-4d5d-8c59-60b8e6f89475/0d6bced7-1bbd-4604-8bae-89d93aa4735e"
-					(reference "#PWR02")
+					(reference "#PWR0102")
 					(unit 1)
 				)
@@
 		(on_board yes)
 		(dnp no)
-		(property "Reference" "#PWR07"
+		(property "Reference" "#PWR0105"
 			(at 134.62 81.28 0)
 			(effects
@@
 			(project "OVERALL"
 				(path "/0e81c85d-86ab-4d5d-8c59-60b8e6f89475/0d6bced7-1bbd-4604-8bae-89d93aa4735e"
-					(reference "#PWR07")
+					(reference "#PWR0105")
 					(unit 1)
 				)
@@
 		(on_board yes)
 		(dnp no)
-		(property "Reference" "RV"
+		(property "Reference" "RV2"
 			(at 236.22 44.196 90)
 			(effects
@@
 			(project "OVERALL"
 				(path "/0e81c85d-86ab-4d5d-8c59-60b8e6f89475/0d6bced7-1bbd-4604-8bae-89d93aa4735e"
-					(reference "RV")
+					(reference "RV2")
 					(unit 1)
 				)
@@
 		(on_board yes)
 		(dnp no)
-		(property "Reference" "#PWR06"
+		(property "Reference" "#PWR0110"
 			(at 72.39 25.4 0)
 			(effects
@@
 			(project "OVERALL"
 				(path "/0e81c85d-86ab-4d5d-8c59-60b8e6f89475/0d6bced7-1bbd-4604-8bae-89d93aa4735e"
-					(reference "#PWR06")
+					(reference "#PWR0110")
 					(unit 1)
 				)
@@
 		(dnp no)
 		(fields_autoplaced yes)
-		(property "Reference" "#PWR04"
+		(property "Reference" "#PWR0106"
 			(at 127 88.9 0)
 			(effects
@@
 			(project "OVERALL"
 				(path "/0e81c85d-86ab-4d5d-8c59-60b8e6f89475/0d6bced7-1bbd-4604-8bae-89d93aa4735e"
-					(reference "#PWR04")
-					(unit 1)
-				)
+					(reference "#PWR0106")
+					(unit 1)
+				)

Commit message: finally completed the schematic
Parts:
- removed J4: Conn_01x04_Pin, symbol Connector:Conn_01x04_Pin
- added J19, J22: Conn_01x02, symbol Connector_Generic:Conn_01x02
- added J21: Conn_01x04, symbol Connector_Generic:Conn_01x04
- renumbered C1 to C58, C4 to C59, C3 to C60, C2 to C61, C7 to C62, C9 to C63, C8 to C64, C5 to C65, C6 to C66, D1 to D8, J2 to J20, J1 to J23, J3 to J24, L1 to L5, L2 to L6, R1 to R51, R6 to R52, R5 to R53, R2 to R54, R3 to R55, R4 to R56, RV2 to RV1, RV1 to RV2, U1 to U14
Connections:
- net +3V3: no longer A1.36 (3V3)
- net GND: now also J19.2 (Pin_2), J21.2 (Pin_2), J22.2 (Pin_2)
- net USB_DM: now also J21.3 (Pin_3)
- net USB_DP: now also J21.4 (Pin_4)
- net 5V: now reaches A1.40 (VBUS)
- net 5V: now also J21.1 (Pin_1)
- net VIN renamed VBAT
- net VBAT: now also J19.1 (Pin_1), J22.1 (Pin_1)
- no-connect marks 5 -> 8
Other:
- note added: "BOOST CONVERTER"
- note added: "BREAKOUT HEADER"
- note added: "BUCK CONVERTER"
- note added: "CIPHER - by ARYAN-GIT-BYTE"
- note added: "MCU"
- note added: "PI PICO 1 BASED ON RP2040"
- moved on the sheet: A1, J24

Commit message: DOCUMENTED Till the Navigation board
Parts:
- removed J21: Conn_01x04, symbol Connector_Generic:Conn_01x04
- added J21, J60: Conn_01x02, symbol Connector_Generic:Conn_01x02
Connections:
- net 5V: now also J21.1 (Pin_1)
- net GND: now also J21.2 (Pin_2)
- net USB_DM: now also J60.1 (Pin_1)
- net USB_DP: now also J60.2 (Pin_2)
Other:
- moved on the sheet: A1

Commit message: changed buck converters
Parts:
- added J59: Screw_Terminal_01x02, symbol Connector:Screw_Terminal_01x02
- added U12: SP3485EP, Package_DIP:DIP-8_W7.62mm, symbol Interface_UART:SP3485EP
- C63, C64: value 12uF -> 22uF
- L6: value 2 uH -> 10 uH
Connections:
- net P16: now also U12.1 (RO)
- net P17: now also U12.2 (~{RE})
- net P18: now also U12.3 (DE)
- net P19: now also U12.4 (DI)
- new net: J59.1 (Pin_1), U12.6 (A)
- new net: J59.2 (Pin_2), U12.7 (B)
Changed lines of the file:
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@@
 	(rectangle
 		(start 20.32 16.51)
-		(end 129.54 114.3)
+		(end 135.89 114.3)
 		(stroke
 			(width 0)
@@
 	)
 	(rectangle
-		(start 140.97 68.58)
+		(start 137.16 67.31)
 		(end 281.94 120.65)
 		(stroke
@@
 	(wire
 		(pts
+			(xy 114.3 57.15) (xy 115.57 57.15)
+		)
+		(stroke
+			(width 0)
+			(type default)
+		)
+	)
+	(wire
+		(pts
 			(xy 78.74 41.91) (xy 86.36 41.91)
 		)
@@
 	(wire
 		(pts
+			(xy 115.57 53.34) (xy 115.57 52.07)
+		)
+		(stroke
+			(width 0)
+			(type default)
+		)
+	)
+	(wire
+		(pts
 			(xy 27.94 74.93) (xy 33.02 74.93)
 		)
@@
 	(wire
 		(pts
+			(xy 91.44 64.77) (xy 91.44 62.23)
+		)
+		(stroke
+			(width 0)
+			(type default)
+		)
+	)
+	(wire
+		(pts
 			(xy 57.15 142.24) (xy 71.12 142.24)
 		)
@@
 	(wire
 		(pts
-			(xy 83.82 57.15) (xy 78.74 57.15)
+			(xy 78.74 57.15) (xy 93.98 57.15)
 		)
 		(stroke
@@
 	(wire
 		(pts
-			(xy 83.82 59.69) (xy 78.74 59.69)
+			(xy 78.74 59.69) (xy 93.98 59.69)
 		)
 		(stroke
@@
 	(wire
 		(pts
-			(xy 83.82 54.61) (xy 78.74 54.61)
+			(xy 78.74 54.61) (xy 93.98 54.61)
 		)
 		(stroke
@@
 	(wire
 		(pts
-			(xy 83.82 62.23) (xy 78.74 62.23)
+			(xy 115.57 52.07) (xy 114.3 52.07)
+		)
+		(stroke
+			(width 0)
+			(type default)
+		)
+	)
+	(wire
+		(pts
+			(xy 116.84 53.34) (xy 115.57 53.34)
+		)
+		(stroke
+			(width 0)
+			(type default)
+		)
+	)
+	(wire
+		(pts
+			(xy 78.74 62.23) (xy 91.44 62.23)
 		)
 		(stroke
@@
 	(wire
 		(pts
+			(xy 115.57 57.15) (xy 115.57 55.88)
+		)
+		(stroke
+			(width 0)
+			(type default)
+		)
+	)
+	(wire
+		(pts
 			(xy 245.11 38.1) (xy 245.11 41.91)
 		)
@@
 	(wire
 		(pts
+			(xy 91.44 64.77) (xy 93.98 64.77)
+		)
+		(stroke
+			(width 0)
+			(type default)
+		)
+	)
+	(wire
+		(pts
 			(xy 57.15 134.62) (xy 71.12 134.62)
 		)
@@
 	(wire
 		(pts
+			(xy 115.57 55.88) (xy 116.84 55.88)
+		)
+		(stroke
+			(width 0)
+			(type default)
+		)
+	)
+	(wire
+		(pts
 			(xy 27.94 54.61) (xy 33.02 54.61)
 		)
@@
 	)
 	(symbol
+		(lib_id "Interface_UART:SP3485EP")
+		(at 104.14 59.69 0)
+		(unit 1)
+		(exclude_from_sim no)
+		(in_bom yes)
+		(on_board yes)
+		(dnp no)
+		(fields_autoplaced yes)
+		(property "Reference" "U12"
+			(at 106.2833 41.91 0)
+			(effects
+				(font
+					(size 1.27 1.27)
+				)
+				(justify left)
+			)
+		)
+		(property "Value" "SP3485EP"
+			(at 106.2833 44.45 0)
+			(effects
+				(font
+					(size 1.27 1.27)
+				)
+				(justify left)
+			)
+		)
+		(property "Footprint" "Package_DIP:DIP-8_W7.62mm"
+			(at 104.14 59.69 0)
+			(effects
+				(font
+					(size 1.27 1.27)
+					(italic yes)
+				)
+				(hide yes)
+			)
+		)
+		(property "Datasheet" "http://www.icbase.com/pdf/SPX/SPX00480106.pdf"
+			(at 104.14 59.69 0)
+			(effects
+				(font
+					(size 1.27 1.27)
+				)
+				(hide yes)
+			)
+		)
+		(property "Description" "Industrial 3.3V Low Power Half-Duplex RS-485 Transceiver 10Mbps, DIP8"
+			(at 104.14 59.69 0)
+			(effects
+				(font
+					(size 1.27 1.27)
+				)
+				(hide yes)
+			)
+		)
+		(pin "7"
+		)
+		(pin "2"
+		)
+		(pin "5"
+		)
+		(pin "8"
+		)
+		(pin "4"
+		)
+		(pin "6"
+		)
+		(pin "1"
+		)
+		(pin "3"
+		)
+		(instances
+			(project ""
+				(path "/0e81c85d-86ab-4d5d-8c59-60b8e6f89475/0d6bced7-1bbd-4604-8bae-89d93aa4735e"
+					(reference "U12")
+					(unit 1)
+				)
+			)
+		)
+	)
+	(symbol
 		(lib_id "Connector_Generic:Conn_01x02")
 		(at 144.78 74.93 0)
@@
 			)
 		)
-		(property "Value" "12uF"
+		(property "Value" "22uF"
 			(at 253.492 88.392 0)
 			(effects
@@
 			)
 		)
-		(property "Value" "2 uH"
+		(property "Value" "10 uH"
 			(at 236.22 83.82 90)
 			(effects
@@
 			)
 		)
-		(property "Value" "12uF"
+		(property "Value" "22uF"
 			(at 154.432 88.392 0)
 			(effects
@@
 					(unit 1)
 				)
+			)
+		)
+	)
+	(symbol
+		(lib_id "Connector:Screw_Terminal_01x02")
+		(at 121.92 53.34 0)
+		(unit 1)
+		(exclude_from_sim no)
+		(in_bom yes)
+		(on_board yes)
+		(dnp no)
+		(property "Reference" "J59"
+			(at 124.46 53.3399 0)
+			(effects
+				(font
+					(size 1.27 1.27)
+				)
+				(justify left)
+			)
+		)
+		(property "Value" "Screw_Terminal_01x02"
+			(at 113.284 58.928 0)
+			(effects
+				(font
+					(size 1.27 1.27)
+				)
+				(justify left)
+			)
+		)
+		(property "Footprint" ""
+			(at 121.92 53.34 0)
+			(effects
+				(font
+					(size 1.27 1.27)
+				)
+				(hide yes)
+			)
+		)
+		(property "Datasheet" "~"
+			(at 121.92 53.34 0)
+			(effects
+				(font
+					(size 1.27 1.27)
+				)
+				(hide yes)
+			)
+		)
+		(property "Description" "Generic screw terminal, single row, 01x02, script generated (kicad-library-utils/schlib/autogen/connector/)"
+			(at 121.92 53.34 0)
+			(effects
+				(font
+					(size 1.27 1.27)
+				)
+				(hide yes)
+			)
+		)
+		(pin "1"
+		)
+		(pin "2"
+		)
+		(instances
+			(project ""
+				(path "/0e81c85d-86ab-4d5d-8c59-60b8e6f89475/0d6bced7-1bbd-4604-8bae-89d93aa4735e"
+					(reference "J59")
+					(unit 1)
+				)
