File: kicad/Instrument/Instrument.kicad_sch (KiCad schematic)
At the start: 0 parts

Commit message: finally completed the schematic
Parts:
- added A3: RaspberryPi_Pico2_W, Module:RaspberryPi_Pico_W_SMD, symbol MCU_Module:RaspberryPi_Pico_W_Extensive
- added C67, C68: 47nF, symbol Device:C
- added C69, C70, C71, C72: 100nF, symbol Device:C
- added D95, D96: BAV99, Package_TO_SOT_SMD:SOT-23, symbol Diode:BAV99
- added J29, J30, J32, J34: Conn_Coaxial, symbol Connector:Conn_Coaxial
- added J31: Conn_01x04, symbol Connector_Generic:Conn_01x04
- added J33: Conn_01x10, symbol Connector_Generic:Conn_01x10
- added R57, R59: 100K, symbol Device:R
- added R58, R60: 10K, symbol Device:R
- added R61: 470, symbol Device:R
- added R62: 4.7K, symbol Device:R
- added R63: 1k, symbol Device:R
- added U16: MCP6022, symbol Amplifier_Operational:MCP6022
- added U17: AP2112K-3.3, Package_TO_SOT_SMD:SOT-23-5, symbol Regulator_Linear:AP2112K-3.3
- added U18, U19: TXU0104PWR, TXU0104PWR:SOP65P640X120-14N, symbol TXU0104PWR:TXU0104PWR
Connections:
- new net: C68.1, J32.1 (In), R62.2
- new net: J30.1 (In), R59.2
- new net: C67.1, R61.2, R62.1
- new net: J34.1 (In), R63.2
- new net: J33.2 (Pin_2), U18.2 (A1)
- new net: J33.3 (Pin_3), U18.3 (A2)
- new net: J33.4 (Pin_4), U18.4 (A3)
- new net: J33.5 (Pin_5), U18.5 (A4)
- new net: J33.6 (Pin_6), U19.2 (A1)
- new net: J33.7 (Pin_7), U19.3 (A2)
- new net: J33.8 (Pin_8), U19.4 (A3)
- new net: J33.9 (Pin_9), U19.5 (A4)
- new net: A3.21 (GPIO16), R61.1
- new net: J29.1 (In), R57.2
- new net: A3.5 (GPIO3), U18.10 (B4Y)
- new net: A3.4 (GPIO2), U18.11 (B3Y)
- new net: A3.2 (GPIO1), U18.12 (B2Y)
- new net: A3.1 (GPIO0), U18.13 (B1Y)
- new net: U18.6 (NC), U18.9 (NC)
- new net: A3.10 (GPIO7), U19.10 (B4Y)
- new net: A3.9 (GPIO6), U19.11 (B3Y)
- new net: A3.7 (GPIO5), U19.12 (B2Y)
- new net: A3.6 (GPIO4), U19.13 (B1Y)
- new net: U19.6 (NC), U19.9 (NC)
- new net: A3.34 (GPIO28_ADC2), R63.1
- new net 3.3V: C69.1, C70.1
- new net 3.3V_ANA: A3.35 (ADC_VREF), D95.2 (A), D96.2 (A), U16.8 (V+), U17.5 (VOUT)
- new net 3v3: A3.36 (3V3), U18.14 (VCCB), U18.8 (OE), U19.14 (VCCB), U19.8 (OE)
- new net 5V: A3.40 (VBUS), J31.1 (Pin_1), U17.1 (VIN), U17.3 (EN)
- new net ADC0: A3.31 (GPIO26_ADC0), U16.1, U16.2 (-)
- new net ADC1: A3.32 (GPIO27_ADC1), U16.6 (-), U16.7
- new net CH1_NODE: D95.3 (K), R57.1, R58.2, U16.3 (+)
- new net CH2_NODE: D96.3 (K), R59.1, R60.2, U16.5 (+)
- new net GND: A3.13 (GND), A3.18 (GND), A3.23 (GND), A3.28 (GND), A3.3 (GND), A3.33 (AGND), A3.38 (GND), A3.8 (GND), A3.D2 (GND), A3.TP1 (USB_GND), C67.2, C68.2, C69.2, C70.2, C71.2, C72.2, D95.1 (K), D96.1 (K), J29.2 (Ext), J30.2 (Ext), J31.2 (Pin_2), J32.2 (Ext), J33.10 (Pin_10), J34.2 (Ext), R58.1, R60.1, U16.4 (V-), U17.2 (GND), U18.7 (GND), U19.7 (GND)
- new net USB_DM: A3.TP2 (USB_DM), J31.3 (Pin_3)
- new net USB_DP: A3.TP3 (USB_DP), J31.4 (Pin_4)
- new net VREF: C71.1, C72.1, J33.1 (Pin_1), U18.1 (VCCA), U19.1 (VCCA)
- no-connect marks 0 -> 21
Other:
- note added: "AP2112K"
- note added: "BREAKOUT HEADERS"
- note added: "CH1_NODE"
- note added: "CH2_NODE"
- note added: "PI PICO 2W"
- note added: "TXU0104PWR"

Commit message: DOCUMENTED Till the Navigation board
Parts:
- removed J31: Conn_01x04, symbol Connector_Generic:Conn_01x04
Connections:
- net 3.3V is gone; now on net 3v3: C69.1, C70.1
Changed lines of the file:
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@@
 	)
 	(junction
-		(at 200.66 81.28)
-		(diameter 0)
-		(color 0 0 0 0)
-	)
-	(junction
-		(at 193.04 93.98)
-		(diameter 0)
-		(color 0 0 0 0)
-	)
-	(junction
 		(at 109.22 34.29)
 		(diameter 0)
@@
 	)
 	(junction
-		(at 193.04 91.44)
-		(diameter 0)
-		(color 0 0 0 0)
-	)
-	(junction
 		(at 80.01 171.45)
 		(diameter 0)
@@
 	)
 	(junction
-		(at 194.31 88.9)
-		(diameter 0)
-		(color 0 0 0 0)
-	)
-	(junction
 		(at 163.83 158.75)
 		(diameter 0)
@@
 	(wire
 		(pts
+			(xy 168.91 78.74) (xy 168.91 81.28)
+		)
+		(stroke
+			(width 0)
+			(type default)
+		)
+	)
+	(wire
+		(pts
 			(xy 64.77 142.24) (xy 77.47 142.24)
 		)
@@
 	(wire
 		(pts
-			(xy 168.91 81.28) (xy 173.99 81.28)
-		)
-		(stroke
-			(width 0)
-			(type default)
-		)
-	)
-	(wire
-		(pts
 			(xy 118.11 99.06) (xy 118.11 109.22)
 		)
@@
 	(wire
 		(pts
-			(xy 200.66 86.36) (xy 200.66 81.28)
-		)
-		(stroke
-			(width 0)
-			(type default)
-		)
-	)
-	(wire
-		(pts
 			(xy 116.84 86.36) (xy 113.03 86.36)
 		)
@@
 	(wire
 		(pts
-			(xy 200.66 81.28) (xy 205.74 81.28)
-		)
-		(stroke
-			(width 0)
-			(type default)
-		)
-	)
-	(wire
-		(pts
 			(xy 232.41 58.42) (xy 232.41 52.07)
 		)
@@
 	(wire
 		(pts
-			(xy 163.83 76.2) (xy 163.83 81.28)
+			(xy 173.99 78.74) (xy 168.91 78.74)
 		)
 		(stroke
@@
 	(wire
 		(pts
-			(xy 200.66 76.2) (xy 163.83 76.2)
+			(xy 163.83 77.47) (xy 163.83 81.28)
 		)
 		(stroke
@@
 		)
 	)
-	(wire
+	(polyline
 		(pts
-			(xy 201.93 86.36) (xy 200.66 86.36)
+			(xy 173.99 163.83) (xy 173.99 181.61)
 		)
 		(stroke
@@
 	(wire
 		(pts
-			(xy 201.93 93.98) (xy 193.04 93.98)
-		)
-		(stroke
-			(width 0)
-			(type default)
-		)
-	)
-	(polyline
-		(pts
-			(xy 173.99 163.83) (xy 173.99 181.61)
+			(xy 163.83 77.47) (xy 165.1 77.47)
 		)
 		(stroke
@@
 	(wire
 		(pts
-			(xy 194.31 88.9) (xy 201.93 88.9)
-		)
-		(stroke
-			(width 0)
-			(type default)
-		)
-	)
-	(wire
-		(pts
 			(xy 177.8 31.75) (xy 193.04 31.75)
 		)
@@
 	(wire
 		(pts
-			(xy 200.66 81.28) (xy 200.66 76.2)
-		)
-		(stroke
-			(width 0)
-			(type default)
-		)
-	)
-	(wire
-		(pts
 			(xy 217.17 106.68) (xy 229.87 106.68)
 		)
@@
 	(wire
 		(pts
-			(xy 201.93 91.44) (xy 193.04 91.44)
-		)
-		(stroke
-			(width 0)
-			(type default)
-		)
-	)
-	(wire
-		(pts
 			(xy 217.17 34.29) (xy 232.41 34.29)
 		)
@@
 		)
 	)
+	(label "3v3"
+		(at 83.82 163.83 180)
+		(effects
+			(font
+				(size 1.27 1.27)
+			)
+			(justify right bottom)
+		)
+	)
+	(label "3v3"
+		(at 173.99 78.74 180)
+		(effects
+			(font
+				(size 1.27 1.27)
+			)
+			(justify right bottom)
+		)
+	)
 	(label "VREF"
 		(at 66.04 111.76 180)
@@
 		)
 	)
-	(label "3v3"
-		(at 173.99 81.28 180)
-		(effects
-			(font
-				(size 1.27 1.27)
-			)
-			(justify right bottom)
-		)
-	)
 	(label "ADC0"
 		(at 195.58 132.08 180)
@@
 		)
 	)
-	(hierarchical_label "3.3V"
+	(hierarchical_label "5V"
 		(shape bidirectional)
-		(at 83.82 163.83 0)
+		(at 165.1 77.47 0)
 		(effects
 			(font
@@
 	(hierarchical_label "5V"
 		(shape bidirectional)
-		(at 205.74 81.28 0)
-		(effects
-			(font
-				(size 1.27 1.27)
-			)
-			(justify left)
-		)
-	)
-	(hierarchical_label "5V"
-		(shape bidirectional)
 		(at 104.14 34.29 180)
 		(effects
@@
 					(unit 1)
 				)
-			)
-		)
-	)
-	(symbol
-		(lib_id "Connector_Generic:Conn_01x04")
-		(at 207.01 88.9 0)
-		(unit 1)
-		(exclude_from_sim no)
-		(in_bom yes)
-		(on_board yes)
-		(dnp no)
-		(fields_autoplaced yes)
-		(property "Reference" "J31"
-			(at 209.55 88.8999 0)
-			(effects
-				(font
-					(size 1.27 1.27)
-				)
-				(justify left)
-			)
-		)
-		(property "Value" "Conn_01x04"
-			(at 209.55 91.4399 0)
-			(effects
-				(font
-					(size 1.27 1.27)
-				)
-				(justify left)
-			)
-		)
-		(property "Footprint" ""
-			(at 207.01 88.9 0)
-			(effects
-				(font
-					(size 1.27 1.27)
-				)
-				(hide yes)
-			)
-		)
-		(property "Datasheet" "~"
-			(at 207.01 88.9 0)
-			(effects
-				(font
-					(size 1.27 1.27)
-				)
-				(hide yes)
-			)
-		)
-		(property "Description" "Generic connector, single row, 01x04, script generated (kicad-library-utils/schlib/autogen/connector/)"
-			(at 207.01 88.9 0)
-			(effects
-				(font
-					(size 1.27 1.27)
-				)
-				(hide yes)
-			)
-		)
-		(pin "2"
-		)
-		(pin "3"
-		)
-		(pin "1"
-		)
-		(pin "4"
-		)
-		(instances
-			(project ""
-				(path "/0e81c85d-86ab-4d5d-8c59-60b8e6f89475/e1a52823-f947-4610-9419-62373c9ba07e"
-					(reference "J31")
-					(unit 1)
-				)
