File: kicad/Navigation-Board/Navigation-Board.kicad_sch (KiCad schematic)
At the start: 178 parts, among them J1 2.8" TFT, J2 0.96" OLED, J3 GME0831B, J4 Conn_01x03, SW1 SW_SPST, SW10 SW_SPST, SW11 SW_SPST, SW12 SW_SPST, SW13 SW_SPST, SW14 SW_SPST, SW15 SW_SPST, SW16 SW_SPST, SW17 SW_SPST, SW18 SW_SPST, SW19 SW_SPST, SW2 SW_SPST, SW20 SW_SPST, SW21 SW_SPST, SW22 SW_SPST, SW23 SW_SPST, SW24 SW_SPST, SW25 SW_SPST, SW26 SW_SPST, SW27 SW_SPST, SW28 SW_SPST, SW29 SW_SPST, SW3 SW_SPST, SW30 SW_SPST, SW31 SW_SPST, SW32 SW_SPST, SW33 SW_SPST, SW34 SW_SPST, SW35 SW_SPST, SW36 SW_SPST, SW37 SW_SPST, SW38 SW_SPST, SW39 SW_SPST, SW4 SW_SPST, SW40 SW_SPST, SW41 SW_SPST, SW42 SW_SPST, SW43 SW_SPST, SW44 SW_SPST, SW45 SW_SPST, SW46 SW_SPST, SW47 SW_SPST, SW48 SW_SPST, SW49 SW_SPST, SW5 SW_SPST, SW50 SW_SPST, SW51 SW_SPST, SW52 SW_SPST, SW53 SW_SPST, SW54 SW_SPST, SW55 SW_SPST, SW56 SW_SPST, SW57 SW_SPST, SW58 SW_SPST, SW59 SW_SPST, SW6 SW_SPST, SW60 SW_SPST, SW61 SW_SPST, SW62 SW_SPST, SW63 SW_SPST, SW64 SW_SPST, SW65 SW_SPST, SW66 SW_SPST, SW67 SW_SPST, SW68 SW_SPST, SW69 SW_SPST, SW7 SW_SPST, SW70 SW_SPST, SW71 SW_SPST, SW72 SW_SPST, SW73 SW_SPST, SW74 SW_SPST, SW75 SW_SPST, SW76 SW_SPST, SW77 SW_SPST, SW78 SW_SPST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

Commit message: made overall schematic
Connections:
- net USB_GND: now reaches A1.TP1 (USB_GND), J4.1 (Pin_1)
- net USB_DM: now reaches A1.TP2 (USB_DM), J4.2 (Pin_2)
- net USB_DP: now reaches A1.TP3 (USB_DP), J4.3 (Pin_3)
Other:
- moved on the sheet: J4

Commit message: finally completed the schematic
Parts:
- renumbered A1 to A2, D2 to D10, D3 to D11, D4 to D12, D5 to D13, D6 to D14, D7 to D15, D8 to D16, D9 to D17, D10 to D18, D11 to D19, D12 to D20, D13 to D21, D14 to D22, D15 to D23, D16 to D24, D17 to D25, D18 to D26, D19 to D27, D20 to D28, D21 to D29, D22 to D30, D23 to D31, D24 to D32, D25 to D33, D26 to D34, D27 to D35, D28 to D36, D29 to D37, D30 to D38, D31 to D39, D32 to D40, D33 to D41, D34 to D42, D35 to D43, D36 to D44, D37 to D45, D38 to D46, D39 to D47, D40 to D48, D41 to D49, D42 to D50, D43 to D51, D44 to D52, D45 to D53, D46 to D54, D47 to D55, D48 to D56, D49 to D57, D50 to D58, D51 to D59, D52 to D60, D53 to D61, D54 to D62, D55 to D63, D56 to D64, D57 to D65, D58 to D66, D59 to D67, D60 to D68, D61 to D69, D62 to D70, D63 to D71, D64 to D72, D65 to D73, D66 to D74, D67 to D75, D68 to D76, D69 to D77, D70 to D78, D71 to D79, D72 to D80, D73 to D81, D74 to D82, D75 to D83, D76 to D84, D77 to D85, D78 to D86, D79 to D87, D80 to D88, D81 to D89, D1 to D9, D82 to D90, D83 to D91, D84 to D92, D86 to D93, D85 to D94, J1 to J25, J2 to J26, J4 to J27, J3 to J28, SW9 to SW10, SW10 to SW11, SW11 to SW12, SW12 to SW13, SW13 to SW14, SW14 to SW15, SW15 to SW16, SW16 to SW17, SW17 to SW18, SW18 to SW19, SW1 to SW2, SW19 to SW20, SW20 to SW21, SW21 to SW22, SW22 to SW23, SW23 to SW24, SW24 to SW25, SW25 to SW26, SW26 to SW27, SW27 to SW28, SW28 to SW29, SW2 to SW3, SW29 to SW30, SW30 to SW31, SW31 to SW32, SW32 to SW33, SW33 to SW34, SW34 to SW35, SW35 to SW36, SW36 to SW37, SW37 to SW38, SW38 to SW39, SW3 to SW4, SW39 to SW40, SW40 to SW41, SW41 to SW42, SW42 to SW43, SW43 to SW44, SW44 to SW45, SW45 to SW46, SW46 to SW47, SW47 to SW48, SW48 to SW49, SW4 to SW5, SW49 to SW50, SW50 to SW51, SW51 to SW52, SW52 to SW53, SW53 to SW54, SW54 to SW55, SW55 to SW56, SW56 to SW57, SW57 to SW58, SW58 to SW59, SW5 to SW6, SW59 to SW60, SW60 to SW61, SW61 to SW62, SW62 to SW63, SW63 to SW64, SW64 to SW65, SW65 to SW66, SW66 to SW67, SW67 to SW68, SW68 to SW69, SW6 to SW7, SW69 to SW70, SW70 to SW71, SW71 to SW72, SW72 to SW73, SW73 to SW74, SW74 to SW75, SW75 to SW76, SW76 to SW77, SW77 to SW78, SW78 to SW79, SW7 to SW8, SW79 to SW80, SW80 to SW81, SW81 to SW82, SW82 to SW83, SW83 to SW84, SW84 to SW85, SW85 to SW86, SW86 to SW87, SW8 to SW9, U1 to U15
Connections:
- net CLK is gone; now on net SCK: A2.24 (GPIO18)
- net SCL: now also J26.4 (Pin_4), J28.4 (Pin_4), U15.22 (SCL); no longer A2.20 (GPIO15)
- removed net SDA: A2.19 (GPIO14), J26.4 (Pin_4), J28.4 (Pin_4), U15.22 (SCL)
- no-connect marks 9 -> 13

Commit message: DOCUMENTED Till the Navigation board
Parts:
- removed J27: Conn_01x03, symbol Connector_Generic:Conn_01x03
- added J27: Conn_01x02, symbol Connector_Generic:Conn_01x02
- added J31: Conn_01x04, symbol Connector_Generic:Conn_01x04
Connections:
- net GND: now also J27.2 (Pin_2)
- net SCL: now also A2.20 (GPIO15), J31.1 (Pin_1); no longer J26.4 (Pin_4), J28.4 (Pin_4), U15.22 (SCL)
- net USB_DM: now also J31.3 (Pin_3)
- net USB_DP: now also J31.4 (Pin_4)
- net SDA: now reaches A2.19 (GPIO14)
- net SDA: now also J26.4 (Pin_4), J28.4 (Pin_4), U15.22 (SCL), J31.2 (Pin_2)
- net 5V: now reaches A2.40 (VBUS)
- net 5V: now also J27.1 (Pin_1)
- net USB_GND: no longer names the net of A2.TP1 (USB_GND)
- no-connect marks 13 -> 10
