File: kicad/Navigation-Board/Navigation-Board.kicad_sch (KiCad schematic)
At the start: 11 parts, among them J1 2.8" TFT, J2 0.96" OLED, J3 Conn_01x04, J4 GME0831B, J5 Conn_01x02, J6 Conn_02x05_Odd_Even, U1 PCA9555D, U2 ESP32-S3-WROOM-1U-N16R8

Commit message: Updated Navigation Board
Parts:
- removed D1, D2: D, Diode_THT:D_DO-35_SOD27_P7.62mm_Horizontal, symbol Device:D
- removed J5: Conn_01x02, symbol Connector_Generic:Conn_01x02
- removed J6: Conn_02x05_Odd_Even, symbol Connector_Generic:Conn_02x05_Odd_Even
- removed U2: ESP32-S3-WROOM-1U-N16R8, RF_Module:ESP32-S3-WROOM-1U, symbol RF_Module:ESP32-S3-WROOM-1
- added A2: RaspberryPi_Pico, Module:RaspberryPi_Pico_SMD, symbol MCU_Module:RaspberryPi_Pico_Extensive
- added C1: 100 nF, symbol Device:C
- added C2: 100nF, symbol Device:C
- added R1, R2: 4.7K, symbol Device:R
- added SW91, SW92, SW93: RotaryEncoder_Switch_MP, symbol Device:RotaryEncoder_Switch_MP
- added U2: 24LC256, symbol Memory_EEPROM:24LC256
Connections:
- net +3V3: now also RV1.1, U1.24 (VDD), A2.36 (3V3), C1.2, C2.1, R1.1, R2.1, U2.8 (VCC); no longer J1.8 (Pin_8)
- net CS: now also A2.17 (GPIO13)
- net DC: now also A2.27 (GPIO21)
- net GND: now also J3.2 (Pin_2), RV1.3, U1.12 (VSS), U1.2 (A1), U1.21 (A0), U1.3 (A2), A2.13 (GND), A2.18 (GND), A2.23 (GND), A2.28 (GND), A2.3 (GND), A2.33 (AGND), A2.38 (GND), A2.8 (GND), A2.D2 (GND), A2.TP1 (USB_GND), C1.1, C2.2, SW91.C, SW91.MP, SW91.S2, SW92.C, SW92.MP, SW92.S2, SW93.C, SW93.MP, U2.1 (A0), U2.2 (A1), U2.3 (A2), U2.4 (GND), U2.7 (WP)
- net MISO: now also A2.21 (GPIO16)
- net MOSI: now also A2.25 (GPIO19)
- net RST: now also A2.29 (GPIO22)
- net SCK: now also A2.24 (GPIO18)
- net SCL: now also U1.23 (SDA), A2.20 (GPIO15), R2.2, U2.6 (SCL); no longer J3.1 (Pin_1)
- net SDA: now also U1.22 (SCL), A2.19 (GPIO14), R1.2, U2.5 (SDA); no longer J3.2 (Pin_2)
- net Switches/C1: now also U1.4 (IO0_0)
- net Switches/C2: now also U1.5 (IO0_1)
- net Switches/C3: now also U1.6 (IO0_2)
- net Switches/C4: now also U1.7 (IO0_3)
- net Switches/R1: now also A2.1 (GPIO0)
- net Switches/R2: now also A2.2 (GPIO1)
- net Switches/R3: now also A2.4 (GPIO2)
- net Switches/R4: now also A2.5 (GPIO3)
- net Switches/R5: now also A2.6 (GPIO4)
- net Switches/R6: now also A2.7 (GPIO5)
- net Switches/R7: now also A2.9 (GPIO6)
- net Switches/R8: now also A2.10 (GPIO7)
- net Switches/R9: now also A2.11 (GPIO8)
- net T_CS: now also A2.22 (GPIO17)
- net T_IRQ: now also A2.26 (GPIO20)
- net USB_DM: now also A2.TP2 (USB_DM)
- net USB_DP: now also A2.TP3 (USB_DP)
- net A0: now reaches RV1.2
- net A0: now also A2.31 (GPIO26_ADC0)
- net PCA9555D_INT: now reaches U1.1 (~{INT})
- net PCA9555D_INT: now also A2.15 (GPIO11)
- net Switches/C7: now reaches U1.10 (IO0_6)
- net Switches/C8: now reaches U1.11 (IO0_7)
- net Switches/C9: now reaches U1.13 (IO1_0)
- net Switches/C10: now reaches U1.14 (IO1_1)
- net E1_S1: now reaches U1.15 (IO1_2)
- net E1_S1: now also SW91.S1
- net E2_S1: now reaches U1.16 (IO1_3)
- net E2_S1: now also SW92.S1
- net E1_A: now reaches U1.17 (IO1_4)
- net E1_A: now also SW91.A
- net E1_B: now reaches U1.18 (IO1_5)
- net E1_B: now also SW91.B
- net E2_A: now reaches U1.19 (IO1_6)
- net E2_A: now also SW92.A
- net E2_B: now reaches U1.20 (IO1_7)
- net E2_B: now also SW92.B
- net Switches/C5: now reaches U1.8 (IO0_4)
- net Switches/C6: now reaches U1.9 (IO0_5)
- net P11 renamed GT911_RST
- net GT911_RST: now also A2.12 (GPIO9)
- net P12 renamed GT911_INT
- net GT911_INT: now also A2.14 (GPIO10)
- new net +5V: A2.40 (VBUS), J3.1 (Pin_1)
- new net E3_A: A2.32 (GPIO27_ADC1), SW93.A
- new net E3_B: A2.34 (GPIO28_ADC2), SW93.B
- new net LED: A2.16 (GPIO12), J1.8 (Pin_8)
Other:
- sheet Switches ports: added C10, C5, C6, C7, C8, C9; removed none
- note added: "CONNECTOR"
- note added: "DISPLAYs"
- note added: "EEPROM"
- note added: "ENCODERs"
- note added: "GPIO EXPANDER"
- note added: "LINEAR POTENTIOMETER"
- note added: "MCU"
- note added: "TOUCHPAD"
- note removed: "DISPLAYS"
- note removed: "MCU & GPIO EXPANDER"
- note removed: "ROTARIES"
- note removed: "TFT FOR MACROPAD/WIDGETS & OLED FOR SYSTEM INFO"
- note removed: "TOUCH PANEL FOR TRACKPAD"
- moved on the sheet: J1, J2, J4, RV1, U1
