File: kicad/OVERALL/OVERALL.kicad_sch (KiCad schematic)
At the start: 0 parts

Commit message: worked on main board
Other:
- sheet GPIO breakout board: file /home/aryan-kumar/Projects/CIPHER/kicad/GPIO-board/GPIO-board.kicad_sch -> ../GPIO-board/GPIO-board.kicad_sch
- sheet Instrument board: file /home/aryan-kumar/Projects/CIPHER/kicad/Instrument/Instrument.kicad_sch -> ../Instrument/Instrument.kicad_sch
- sheet Main-Board: file /home/aryan-kumar/Projects/CIPHER/kicad/main-board/main-board.kicad_sch -> ../main-board/main-board.kicad_sch
- sheet Navigation Board: file /home/aryan-kumar/Projects/CIPHER/kicad/Navigation-Board/Navigation-Board.kicad_sch -> ../Navigation-Board/Navigation-Board.kicad_sch
- sheet Power Board: file /home/aryan-kumar/Projects/CIPHER/kicad/power-supply/power-supply.kicad_sch -> ../power-supply/power-supply.kicad_sch
Changed lines of the file:
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@@
 			)
 		)
-		(property "Sheetfile" "/home/aryan-kumar/Projects/CIPHER/kicad/GPIO-board/GPIO-board.kicad_sch"
+		(property "Sheetfile" "../GPIO-board/GPIO-board.kicad_sch"
 			(at 210.82 116.1546 0)
 			(effects
@@
 			)
 		)
-		(property "Sheetfile" "/home/aryan-kumar/Projects/CIPHER/kicad/power-supply/power-supply.kicad_sch"
+		(property "Sheetfile" "../power-supply/power-supply.kicad_sch"
 			(at 26.924 114.3 0)
 			(effects
@@
 			)
 		)
-		(property "Sheetfile" "/home/aryan-kumar/Projects/CIPHER/kicad/main-board/main-board.kicad_sch"
+		(property "Sheetfile" "../main-board/main-board.kicad_sch"
 			(at 119.38 116.1546 0)
 			(effects
@@
 			)
 		)
-		(property "Sheetfile" "/home/aryan-kumar/Projects/CIPHER/kicad/Navigation-Board/Navigation-Board.kicad_sch"
+		(property "Sheetfile" "../Navigation-Board/Navigation-Board.kicad_sch"
 			(at 120.65 159.3346 0)
 			(effects
@@
 			)
 		)
-		(property "Sheetfile" "/home/aryan-kumar/Projects/CIPHER/kicad/Instrument/Instrument.kicad_sch"
+		(property "Sheetfile" "../Instrument/Instrument.kicad_sch"
 			(at 156.21 78.0546 0)
 			(effects

Commit message: update
Other:
- added sheet Radio Board (../Radio-Board/Radio-Board.kicad_sch)
Changed lines of the file:
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@@
+	)
+	(sheet
+		(at 87.63 50.8)
+		(size 43.18 22.86)
+		(exclude_from_sim no)
+		(in_bom yes)
+		(on_board yes)
+		(dnp no)
+		(fields_autoplaced yes)
+		(stroke
+			(width 0.1524)
+			(type solid)
+		)
+		(fill
+			(color 0 0 0 0.0000)
+		)
+		(property "Sheetname" "Radio Board"
+			(at 87.63 50.0884 0)
+			(effects
+				(font
+					(size 1.27 1.27)
+				)
+				(justify left bottom)
+			)
+		)
+		(property "Sheetfile" "../Radio-Board/Radio-Board.kicad_sch"
+			(at 87.63 74.2446 0)
+			(effects
+				(font
+					(size 1.27 1.27)
+				)
+				(justify left top)
+			)
+		)
+		(instances
+			(project "OVERALL"
+				(path "/0e81c85d-86ab-4d5d-8c59-60b8e6f89475"
+					(page "8")
+				)
+			)
+		)
 	)
 	(sheet

Commit message: updated the main board, changes journaled in the fallout journaling
Other:
- sheet Main-Board ports: added USB-DM1, USB-DM2, USB-DP1, USB-DP2; removed none
Changed lines of the file:
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@@
+	(wire
+		(pts
+			(xy 167.64 105.41) (xy 210.82 105.41)
+		)
+		(stroke
+			(width 0)
+			(type default)
+		)
+	)
+	(wire
+		(pts
+			(xy 167.64 107.95) (xy 210.82 107.95)
+		)
+		(stroke
+			(width 0)
+			(type default)
+		)
+	)
 	(wire
 		(pts
@@
 	(wire
 		(pts
+			(xy 152.4 115.57) (xy 152.4 129.54)
+		)
+		(stroke
+			(width 0)
+			(type default)
+		)
+	)
+	(wire
+		(pts
 			(xy 218.44 115.57) (xy 218.44 127)
 		)
@@
 		(pts
 			(xy 214.63 115.57) (xy 214.63 124.46)
+		)
+		(stroke
+			(width 0)
+			(type default)
+		)
+	)
+	(wire
+		(pts
+			(xy 149.86 115.57) (xy 149.86 129.54)
 		)
 		(stroke
@@
 		(on_board yes)
 		(dnp no)
-		(fields_autoplaced yes)
 		(stroke
 			(width 0.1524)
@@
 		)
 		(property "Sheetfile" "../main-board/main-board.kicad_sch"
-			(at 119.38 116.1546 0)
+			(at 121.92 100.33 0)
 			(effects
 				(font
@@
 			)
 		)
+		(pin "USB-DM1" bidirectional
+			(at 152.4 115.57 270)
+			(effects
+				(font
+					(size 1.27 1.27)
+				)
+				(justify left)
+			)
+		)
+		(pin "USB-DP1" bidirectional
+			(at 149.86 115.57 270)
+			(effects
+				(font
+					(size 1.27 1.27)
+				)
+				(justify left)
+			)
+		)
+		(pin "USB-DM2" bidirectional
+			(at 167.64 107.95 0)
+			(effects
+				(font
+					(size 1.27 1.27)
+				)
+				(justify right)
+			)
+		)
+		(pin "USB-DP2" bidirectional
+			(at 167.64 105.41 0)
+			(effects
+				(font
+					(size 1.27 1.27)
+				)
+				(justify right)
+			)
+		)

Commit message: Completed the main board schematic
Other:
- sheet Main-Board ports: added SSD_3V; removed none
Changed lines of the file:
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@@
+	)
+	(junction
+		(at 107.95 127)
+		(diameter 0)
+		(color 0 0 0 0)
 	)
 	(junction
@@
 	(wire
 		(pts
+			(xy 107.95 104.14) (xy 107.95 127)
+		)
+		(stroke
+			(width 0)
+			(type default)
+		)
+	)
+	(wire
+		(pts
 			(xy 76.2 114.3) (xy 76.2 127)
 		)
@@
 	(wire
 		(pts
+			(xy 107.95 127) (xy 76.2 127)
+		)
+		(stroke
+			(width 0)
+			(type default)
+		)
+	)
+	(wire
+		(pts
 			(xy 78.74 93.98) (xy 119.38 93.98)
 		)
@@
 	(wire
 		(pts
-			(xy 218.44 127) (xy 76.2 127)
+			(xy 218.44 127) (xy 107.95 127)
 		)
 		(stroke
@@
 		(pts
 			(xy 149.86 115.57) (xy 149.86 129.54)
+		)
+		(stroke
+			(width 0)
+			(type default)
+		)
+	)
+	(wire
+		(pts
+			(xy 119.38 104.14) (xy 107.95 104.14)
 		)
 		(stroke
@@
 			)
 		)
+		(pin "SSD_3V" input
+			(at 119.38 104.14 180)
+			(effects
+				(font
+					(size 1.27 1.27)
+				)
+				(justify left)
+			)
+		)

Commit message: finally completed the schematic
Other:
- sheet GPIO breakout board ports: added 5V, VBAT; removed 3V3
- sheet Instrument board ports: added 3.3V, 5V, GND, USB_DM, USB_DP; removed none
- sheet Main-Board ports: added CE0, GPI017, GPIO22, GPIO27, GPIO5, MISO, MOSI, SCK, SCL, SDA, USB-DM3, USB-DM4, USB-DP3, USB-DP4; removed none
- sheet Navigation Board ports: added SCL, SDA; removed none
- sheet Power Board ports: added 3V8_OUT, VBAT; removed none
- sheet Radio Board ports: added +5V, 3.3V, 3.8V, CE0, GND, GPI017, GPIO22, GPIO27, GPIO5, MISO, MOSI, SCK, USBD_M, USBD_P; removed none
- note added: "CIPHER by ARYAN-GIT-BYTE"

Commit message: all data got corrupted bruhh. now , commiting whats left healthy
Other:
- sheet Instrument board ports: added none; removed 3.3V
- sheet Navigation Board ports: added 5V, GND; removed 3V3, USB_GND
- note added: "GPIO BREAKOUT BOARD"
- note added: "INSTRUMENT BOARD"
- note added: "MAIN BOARD"
- note added: "NAVIGATION BOARD"
- note added: "POWER BOARD"
- note added: "RADIO BOARD"

Commit message: upddate
Other:
- sheet Power Board ports: added GPIO, SCL, SDA; removed none
Changed lines of the file:
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@@
 (kicad_sch
-	(version 20250114)
+	(version 20260306)
 	(generator "eeschema")
-	(generator_version "9.0")
+	(generator_version "10.0")
 	(paper "A4")
 	(text "GPIO BREAKOUT BOARD"
@@
 	)
 	(junction
+		(at 140.97 107.95)
+		(diameter 0)
+		(color 0 0 0 0)
+	)
+	(junction
 		(at 97.79 143.51)
+		(diameter 0)
+		(color 0 0 0 0)
+	)
+	(junction
+		(at 144.78 105.41)
 		(diameter 0)
 		(color 0 0 0 0)
@@
 	(wire
 		(pts
+			(xy 78.74 107.95) (xy 140.97 107.95)
+		)
+		(stroke
+			(width 0)
+			(type default)
+		)
+	)
+	(wire
+		(pts
 			(xy 109.22 45.72) (xy 109.22 121.92)
 		)
@@
 	(wire
 		(pts
+			(xy 140.97 107.95) (xy 140.97 151.13)
+		)
+		(stroke
+			(width 0)
+			(type default)
+		)
+	)
+	(wire
+		(pts
 			(xy 132.08 135.89) (xy 95.25 135.89)
 		)
@@
 	(wire
 		(pts
-			(xy 140.97 104.14) (xy 140.97 151.13)
+			(xy 140.97 104.14) (xy 140.97 107.95)
 		)
 		(stroke
@@
 	(wire
 		(pts
+			(xy 144.78 105.41) (xy 144.78 151.13)
+		)
+		(stroke
+			(width 0)
+			(type default)
+		)
+	)
+	(wire
+		(pts
 			(xy 95.25 85.09) (xy 95.25 68.58)
 		)
@@
 	(wire
 		(pts
+			(xy 168.91 39.37) (xy 168.91 64.77)
+		)
+		(stroke
+			(width 0)
+			(type default)
+		)
+	)
+	(wire
+		(pts
 			(xy 87.63 118.11) (xy 95.25 118.11)
 		)
@@
 	(wire
 		(pts
-			(xy 168.91 67.31) (xy 168.91 39.37)
-		)
-		(stroke
-			(width 0)
-			(type default)
-		)
-	)
-	(wire
-		(pts
 			(xy 100.33 123.19) (xy 127 123.19)
 		)
@@
 	(wire
 		(pts
-			(xy 144.78 104.14) (xy 144.78 151.13)
+			(xy 144.78 104.14) (xy 144.78 105.41)
+		)
+		(stroke
+			(width 0)
+			(type default)
+		)
+	)
+	(wire
+		(pts
+			(xy 78.74 105.41) (xy 144.78 105.41)
 		)
 		(stroke
@@
 	(wire
 		(pts
-			(xy 165.1 43.18) (xy 165.1 67.31)
+			(xy 165.1 43.18) (xy 165.1 64.77)
 		)
 		(stroke
@@
 		)
 		(fill
-			(color 0 0 0 0.0000)
+			(color 0 0 0 0)
 		)
 		(property "Sheetname" "GPIO breakout board"
 			(at 185.42 114.8584 0)
+			(show_name no)
+			(do_not_autoplace no)
 			(effects
 				(font
@@
 		(property "Sheetfile" "../GPIO-board/GPIO-board.kicad_sch"
 			(at 185.42 141.5546 0)
+			(show_name no)
+			(do_not_autoplace no)
 			(effects
 				(font
@@
 		)
 		(fill
-			(color 0 0 0 0.0000)
+			(color 0 0 0 0)
 		)
 		(property "Sheetname" "Radio Board"
 			(at 34.29 37.3884 0)
+			(show_name no)
+			(do_not_autoplace no)
 			(effects
 				(font
@@
 		(property "Sheetfile" "../Radio-Board/Radio-Board.kicad_sch"
 			(at 32.766 34.29 0)
+			(show_name no)
+			(do_not_autoplace no)
 			(effects
 				(font
@@
 		)
 		(fill
-			(color 0 0 0 0.0000)
+			(color 0 0 0 0)
 		)
 		(property "Sheetname" "Power Board"
 			(at 43.18 100.8884 0)
+			(show_name no)
+			(do_not_autoplace no)
 			(effects
 				(font
@@
 		(property "Sheetfile" "../power-supply/power-supply.kicad_sch"
 			(at 37.338 150.114 0)
+			(show_name no)
+			(do_not_autoplace no)
 			(effects
 				(font
@@
 		(pin "VBAT" bidirectional
 			(at 78.74 137.16 0)
+			(effects
+				(font
+					(size 1.27 1.27)
+				)
+				(justify right)
+			)
+		)
+		(pin "SDA" bidirectional
+			(at 78.74 105.41 0)
+			(effects
+				(font
+					(size 1.27 1.27)
+				)
+				(justify right)
+			)
+		)
+		(pin "SCL" bidirectional
+			(at 78.74 107.95 0)
+			(effects
+				(font
+					(size 1.27 1.27)
+				)
+				(justify right)
+			)
+		)
+		(pin "GPIO" bidirectional
+			(at 78.74 110.49 0)
 			(effects
 				(font
@@
 		)
 		(fill
-			(color 0 0 0 0.0000)
+			(color 0 0 0 0)
 		)
 		(property "Sheetname" "Main-Board"
 			(at 118.11 62.23 0)
+			(show_name no)
+			(do_not_autoplace no)
 			(effects
 				(font
@@
 		(property "Sheetfile" "../main-board/main-board.kicad_sch"
 			(at 118.11 62.738 0)
+			(show_name no)
+			(do_not_autoplace no)
 			(effects
 				(font
@@
 		)
 		(fill
-			(color 0 0 0 0.0000)
+			(color 0 0 0 0)
 		)
 		(property "Sheetname" "Navigation Board"
 			(at 120.65 150.4184 0)
+			(show_name no)
+			(do_not_autoplace no)
 			(effects
 				(font
@@
 		(property "Sheetfile" "../Navigation-Board/Navigation-Board.kicad_sch"
 			(at 120.65 173.3046 0)
+			(show_name no)
+			(do_not_autoplace no)
 			(effects
 				(font
@@
 		)
 		(fill
-			(color 0 0 0 0.0000)
+			(color 0 0 0 0)
 		)
 		(property "Sheetname" "Instrument board"
 			(at 116.332 20.066 0)
+			(show_name no)
+			(do_not_autoplace no)
 			(effects
 				(font
@@
 		(property "Sheetfile" "../Instrument/Instrument.kicad_sch"
 			(at 106.172 21.082 0)
-			(effects
-				(font
+			(show_name no)
+			(do_not_autoplace no)
+			(effects
+				(font
