File: kicad/Radio-Board/Radio-Board.kicad_sch (KiCad schematic)
At the start: 1 part, among them U8 SIM7600E-H

Commit message: finally completed the schematic
Parts:
- added C73, C78: 100nF, symbol Device:C
- added C74: 470uF, symbol Device:C_Polarized
- added C75: 1000uF, symbol Device:C_Polarized
- added C76: 100nf, symbol Device:C
- added C77: 10uF, symbol Device:C
- added D97: SMF05C, SMF05C:SC70-6, symbol SMF05C:SMF05C
- added J35, J53: Conn_01x04, symbol Connector_Generic:Conn_01x04
- added J36: Conn_01x08, symbol Connector_Generic:Conn_01x08
- added J37: SIM_Card_Shielded, symbol Connector:SIM_Card_Shielded
- added J38, J39, J40, J41: Conn_Coaxial, symbol Connector:Conn_Coaxial
- added J42: Conn_01x02, symbol Connector_Generic:Conn_01x02
- added Q10: 2N3904, Package_TO_SOT_THT:TO-92_Inline, symbol Transistor_BJT:2N3904
- added R64: 1K, symbol Device:R_Small
- added TP13, TP14, TP15, TP16, TP17, TP18, TP19, TP20, TP21, TP22, TP23, TP24, TP25, TP26, TP27, TP28, TP29, TP30, TP31, TP32, TP33, TP34, TP35, TP36, TP37, TP38, TP39, TP40, TP41, TP42, TP43, TP44, TP45, TP46, TP47, TP48, TP49, TP50, TP51, TP52, TP53, TP54: TestPoint, symbol Connector:TestPoint
- added U21: SX1262S915N0S1, symbol Vollgo-SX1262S915N0S1:SX1262S915N0S1
- renumbered U8 to U20
Connections:
- net GND: now also C73.2, C74.2, C75.2, C76.1, C77.2, C78.2, D97.2, J35.2 (Pin_2), J37.5 (GND), J37.SH, J38.2 (Ext), J39.2 (Ext), J40.2 (Ext), J41.2 (Ext), Q10.3 (C), U21.12 (GND), U21.13 (GND), U21.7 (GND), U21.9 (GND)
- net VBAT: now also C73.1, C74.1, C75.1, J35.1 (Pin_1)
- net +5V: now reaches U20.11 (USB_VBUS)
- net +5V: now also J35.3 (Pin_3)
- net USBD_M: now reaches U20.12 (USB_DN)
- net USBD_M: now also J42.1 (Pin_1)
- net USBD_P: now reaches U20.13 (USB_DP)
- net USBD_P: now also J42.2 (Pin_2)
- net at U20.15 (VDD_1V8): now also TP15.1
- net at U20.16 (USB_ID): now also TP53.1
- net DATA: now reaches U20.17 (USIM_DATA)
- net DATA: now also D97.5, J37.7 (I/O)
- net RST: now reaches U20.18 (USIM_RST)
- net RST: now also D97.4, J37.2 (RST)
- net CLK: now reaches U20.19 (USIM_CLK)
- net CLK: now also D97.3, J37.3 (CLK)
- net VDD: now reaches U20.20 (USIM_VDD)
- net VDD: now also C76.2, D97.1, J37.1 (VCC)
- net at U20.27 (SDIO_DATA1): now also TP17.1
- net at U20.28 (SDIO_DATA2): now also TP18.1
- net at U20.29 (SDIO_CMD): now also TP20.1
- net at U20.3 (PWRKEY): now also Q10.1 (E)
- net at U20.30 (SDIO_DATA0): now also TP16.1
- net at U20.31 (SDIO_DATA3): now also TP19.1
- net at U20.32 (SDIO_CLK): now also TP21.1
- net at U20.33 (GPIO3): now also TP28.1
- net at U20.34 (GPIO6): now also TP29.1
- net at U20.35 (HSIC_STROBE): now also TP22.1
- net at U20.36 (HSIC_DATA): now also TP23.1
- net at U20.4 (RESET): now also TP14.1
- net at U20.44 (VDD_AUX): now also TP13.1
- net at U20.45 (ISINK): now also TP47.1
- net at U20.46 (ADC2): now also TP49.1
- net at U20.47 (ADC1): now also TP48.1
- net at U20.48 (SD_DET): now also TP43.1
- net at U20.49 (STATUS): now also TP41.1
- net at U20.50 (GPIO43): now also TP33.1
- net at U20.51 (NETLIGHT): now also TP39.1
- net at U20.52 (GPIO41): now also TP31.1
- net at U20.53 (USIM_DET): now also TP44.1
- net at U20.54 (FLIGHTMODE): now also TP37.1
- net at U20.55 (SCL): now also TP45.1
- net at U20.56 (SDA): now also TP46.1
- net at U20.59 (AUX_ANT): now also J41.1 (In)
- net SPI_CLK: now reaches U20.6 (SPI_CLK)
- net SPI_CLK: now also J53.1 (Pin_1)
- net at U20.66 (RTS): now also TP36.1
- net at U20.67 (CTS): now also TP30.1
- net at U20.68 (RXD): now also TP32.1
- net at U20.69 (RI): now also TP38.1
- net SPI_MISO: now reaches U20.7 (SPI_MISO)
- net SPI_MISO: now also J53.4 (Pin_4)
- net at U20.70 (DCD): now also TP40.1
- net at U20.71 (TXD): now also TP42.1
- net at U20.72 (DTR): now also TP34.1
- net at U20.73 (PCM_OUT): now also TP25.1
- net at U20.74 (PCM_IN): now also TP24.1
- net at U20.75 (PCM_SYNC): now also TP26.1
- net at U20.76 (PCM_CLK): now also TP27.1
- net at U20.79 (GNSS_ANT): now also J40.1 (In)
- net SPI_MOSI: now reaches U20.8 (SPI_MOSI)
- net SPI_MOSI: now also J53.3 (Pin_3)
- net at U20.82 (MAIN_ANT): now also J39.1 (In)
- net at U20.83 (COEX1): now also TP50.1
- net at U20.84 (COEX2): now also TP51.1
- net at U20.85 (BOOT_CFG0): now also TP54.1
- net at U20.86 (COEX3): now also TP52.1
- net at U20.87 (GPIO77): now also TP35.1
- net SPI_CS: now reaches U20.9 (SPI_CS)
- net SPI_CS: now also J53.2 (Pin_2)
- new net: J38.1 (In), U21.14 (ANT)
- new net: Q10.2 (B), R64.1
- new net 3.3V: C77.1, C78.1, J35.4 (Pin_4), U21.6 (VCC)
- new net CE0: J36.1 (Pin_1), U21.5 (NSS)
- new net GPI017: J36.4 (Pin_4), U21.11 (BUSY)
- new net GPIO22: J36.3 (Pin_3), U21.1 (RST)
- new net GPIO27: J36.5 (Pin_5), U21.10 (DIO1)
- new net GPIO5: J36.2 (Pin_2), R64.2
- new net MISO: J36.7 (Pin_7), U21.2 (MISO)
- new net MOSI: J36.6 (Pin_6), U21.3 (MOSI)
- new net SCK: J36.8 (Pin_8), U21.4 (SCK)
- no-connect marks 0 -> 9
Other:
- note added: "CIPHER - by ARYAN-GIT-BYTE"
- note added: "External Collector"
- note added: "LTE module"
- note added: "LoRa Module"
- moved on the sheet: U20

Commit message: DOCUMENTED Till the Navigation board
Parts:
- removed J35: Conn_01x04, symbol Connector_Generic:Conn_01x04
- added J35, J61, J62: Conn_01x02, symbol Connector_Generic:Conn_01x02
Connections:
- net +5V: now also J61.1 (Pin_1)
- net 3.3V: now also J62.1 (Pin_1)
- net GND: now also J35.2 (Pin_2), J61.2 (Pin_2), J62.2 (Pin_2)
- net VBAT: now also J35.1 (Pin_1)
Other:
- note added: "EXTERNAL CONNECTOR"
- note added: "POWER CONNECTORS"
- note removed: "External Collector"

Commit message: upddate
Other:
- moved on the sheet: C77, C78, J35, J36, J38, J61, J62, U21
