File: kicad/main-board/main-board.kicad_sch (KiCad schematic)
At the start: 38 parts, among them J1 Conn_01x02, J10 Conn_01x08, J11 Conn_02x20_Odd_Even, J12 AudioPlug3, J13 FAN_HEADERS, J2 Conn_02x07_Odd_Even, J3 Conn_01x03, J4 Conn_01x03, J5 THD-02-R, J6 Conn_01x03, J7 Conn_01x02, J8 Conn_01x03, J9 Micro_SD_Card_Det, U1 TPD4EUSB30, U2 TPD4EUSB30, U3 CM5108064B, U4 MagJack-A70-112-331N126, U5 RT9742GGJ5, U6 PCM5102A

Commit message: DOCUMENTED Till the Navigation board
Parts:
- removed C1: 100n, Capacitor_SMD:C_0402_1005Metric, symbol Device:C
- removed C2: 10u, Capacitor_SMD:C_0805_2012Metric, symbol Device:C
- removed J3, J4, J6, J8: Conn_01x03, symbol Connector_Generic:Conn_01x03
- removed J5: THD-02-R, Connector_PinHeader_2.54mm:PinHeader_2x02_P2.54mm_Vertical, symbol Connector_Generic:Conn_02x02_Odd_Even
- removed J9: Micro_SD_Card_Det, CM5IO:SDCARD_MOLEX_503398-1892, symbol Connector:Micro_SD_Card_Det2
- removed R3, R4: 470R, Resistor_SMD:R_0402_1005Metric, symbol Device:R
- removed U1, U2: TPD4EUSB30, Package_SON:USON-10_2.5x1.0mm_P0.5mm, symbol CM5IO:TPD4EUSB30
- removed U4: MagJack-A70-112-331N126, CM5IO:TRJG0926HENL, symbol CM5IO:MagJack-A70-112-331N126
- removed U5: RT9742GGJ5, Package_TO_SOT_SMD:SOT-23-5, symbol CM5IO:RT9742GGJ5
- added J54, J55, J56: Conn_01x02, symbol Connector_Generic:Conn_01x02
- added J57: Conn_01x04, symbol Connector_Generic:Conn_01x04
Connections:
- net P0 is gone; now on an unnamed net: U3.97 (CAM_GPIO)
- net P1 is gone; now on an unnamed net: U3.100 (CAM_GPIO1)
- net SCL: now also J57.1 (Pin_1)
- net SDA: now also J57.2 (Pin_2)
- net USB-DM1: now also J57.3 (Pin_3)
- net USB-DM2: now also J56.1 (Pin_1)
- net USB-DM3: now also J54.1 (Pin_1)
- net USB-DP1: now also J57.4 (Pin_4)
- net USB-DP2: now also J56.2 (Pin_2)
- net USB-DP3: now also J54.2 (Pin_2)
- net USB-DP4: now also J55.1 (Pin_1)
- net Ports/USBOTG renamed USBOTG
- new net USB-DM4: J55.2 (Pin_2)
- no-connect marks 12 -> 9
Other:
- added sheet Connectors (connectors.kicad_sch)
- note added: "AUDIO JACK"
- note added: "ETHERNET & SD-CARD"
- note added: "FAN HEADERS"
- note added: "GPIO HEADERS"
- note added: "PORTS"
- note removed: "CM5Lite SDCARD I/F"
- note removed: "Ethernet"
- note removed: "Ethernet POE Protection"
- note removed: "POE Header"
- note removed: "POWER LOAD SWITCH FOR SD CARD"
- moved on the sheet: J10, J11, J13, J2, J7, TP1, TP2
