File: kicad/Navigation-Board/_restore_backup_2026-06-30T21-01-58-557/Navigation-Board.kicad_sch (KiCad schematic)
At the start: 11 parts, among them J1 2.8" TFT, J2 0.96" OLED, J3 Conn_01x04, J4 GME0831B, J5 Conn_01x02, J6 Conn_02x05_Odd_Even, U1 PCA9555D, U2 ESP32-S3-WROOM-1U-N16R8

Commit message: son-ion
Parts:
- removed J6: Conn_02x05_Odd_Even, symbol Connector_Generic:Conn_02x05_Odd_Even
- removed RV1: Linear Potentiometer, symbol Device:R_Potentiometer
- removed U2: ESP32-S3-WROOM-1U-N16R8, RF_Module:ESP32-S3-WROOM-1U, symbol RF_Module:ESP32-S3-WROOM-1
- added A1: RaspberryPi_Pico, Module:RaspberryPi_Pico_SMD, symbol MCU_Module:RaspberryPi_Pico_Extensive
Connections:
- net +3V3: now also U1.24 (VDD), A1.36 (3V3); no longer J1.8 (Pin_8)
- net 5V: now also A1.40 (VBUS)
- net ADC1: now also A1.32 (GPIO27_ADC1)
- net ADC2: now also A1.34 (GPIO28_ADC2)
- net C1: now also U1.4 (IO0_0)
- net C10: now also U1.14 (IO1_1)
- net C11: now also U1.15 (IO1_2)
- net C12: now also U1.16 (IO1_3)
- net C13: now also U1.17 (IO1_4)
- net C14: now also U1.18 (IO1_5)
- net C15: now also U1.19 (IO1_6)
- net C16: now also U1.20 (IO1_7)
- net C2: now also U1.5 (IO0_1)
- net C3: now also U1.6 (IO0_2)
- net C4: now also U1.7 (IO0_3)
- net C5: now also U1.8 (IO0_4)
- net C6: now also U1.9 (IO0_5)
- net C7: now also U1.10 (IO0_6)
- net C8: now also U1.11 (IO0_7)
- net C9: now also U1.13 (IO1_0)
- net CS: now also A1.22 (GPIO17)
- net DC: now also A1.26 (GPIO20)
- net GND: now also U1.12 (VSS), U1.2 (A1), U1.21 (A0), U1.3 (A2), A1.13 (GND), A1.18 (GND), A1.23 (GND), A1.28 (GND), A1.3 (GND), A1.33 (AGND), A1.38 (GND), A1.8 (GND), A1.D2 (GND)
- net INT: now also U1.1 (~{INT}), A1.17 (GPIO13)
- net MISO: now also A1.21 (GPIO16)
- net MOSI: now also A1.25 (GPIO19)
- net P09: now also A1.12 (GPIO9)
- net P10: now also A1.14 (GPIO10)
- net P11: now also A1.15 (GPIO11)
- net P12: now also A1.16 (GPIO12)
- net R1: now also A1.4 (GPIO2)
- net R2: now also A1.5 (GPIO3)
- net R3: now also A1.6 (GPIO4)
- net R4: now also A1.7 (GPIO5)
- net R5: now also A1.9 (GPIO6)
- net R6: now also A1.10 (GPIO7)
- net RST: now also A1.27 (GPIO21)
- net SCK: now also A1.24 (GPIO18)
- net SCL: now also U1.23 (SDA), A1.20 (GPIO15)
- net SDA: now also U1.22 (SCL), A1.19 (GPIO14)
- net T_CS: now also A1.31 (GPIO26_ADC0)
- net T_IRQ: now also A1.29 (GPIO22)
- net USB_DM: now also A1.TP2 (USB_DM)
- net USB_DP: now also A1.TP3 (USB_DP)
- new net LED: A1.11 (GPIO8), J1.8 (Pin_8)
Other:
- sheet Switches ports: added none; removed C1, C2, C3, C4, R1, R2, R3, R4, R5, R6, R7, R8, R9
- moved on the sheet: J1, J2
