File: kicad/Navigation-Board/_restore_backup_2026-06-30T21-21-01-393/Navigation-Board.kicad_sch (KiCad schematic)
At the start: 11 parts, among them J1 2.8" TFT, J2 0.96" OLED, J3 Conn_01x04, J4 GME0831B, J5 Conn_01x02, J6 Conn_02x05_Odd_Even, U1 PCA9555D, U2 ESP32-S3-WROOM-1U-N16R8

Commit message: son-ion
Parts:
- removed RV1: Linear Potentiometer, symbol Device:R_Potentiometer
- removed U2: ESP32-S3-WROOM-1U-N16R8, RF_Module:ESP32-S3-WROOM-1U, symbol RF_Module:ESP32-S3-WROOM-1
- added A1: RaspberryPi_Pico, Module:RaspberryPi_Pico_SMD, symbol MCU_Module:RaspberryPi_Pico_Extensive
Connections:
- net +3V3: now also U1.24 (VDD); no longer J1.8 (Pin_8)
- net C1: now also U1.4 (IO0_0)
- net C10: now also U1.14 (IO1_1)
- net C11: now also U1.15 (IO1_2)
- net C12: now also U1.16 (IO1_3)
- net C13: now also U1.17 (IO1_4)
- net C14: now also U1.18 (IO1_5)
- net C15: now also U1.19 (IO1_6)
- net C16: now also U1.20 (IO1_7)
- net C2: now also U1.5 (IO0_1)
- net C3: now also U1.6 (IO0_2)
- net C4: now also U1.7 (IO0_3)
- net C5: now also U1.8 (IO0_4)
- net C6: now also U1.9 (IO0_5)
- net C7: now also U1.10 (IO0_6)
- net C8: now also U1.11 (IO0_7)
- net C9: now also U1.13 (IO1_0)
- net GND: now also U1.12 (VSS), U1.2 (A1), U1.21 (A0), U1.3 (A2)
- net INT: now also U1.1 (~{INT})
- net SCL: now also U1.23 (SDA)
- net SDA: now also U1.22 (SCL)
- new net: A1.13 (GND), A1.18 (GND), A1.23 (GND), A1.28 (GND), A1.3 (GND), A1.38 (GND), A1.8 (GND), A1.D2 (GND)
- new net LED: J1.8 (Pin_8)
Other:
- sheet Switches ports: added none; removed C1, C2, C3, C4, R1, R2, R3, R4, R5, R6, R7, R8, R9
